File: Tec/HW_Laboratory/Laboratory/control.kicad_sch (KiCad schematic)
At the start: 6 parts, among them J10 SPI, J15 I2C, J16 CONTROL, U11 ch32v006k8u6, U3 74HC595, U8 AT24CS04-SSHM

Commit message: Schematics UPDATE
Parts:
- added C6, C9: 100nF, Capacitor_SMD:C_0603_1608Metric, symbol Device:C
Connections:
- net SDA: now reaches J15.1 (Pin_1)
- net SDA: now also U11.14 (PC1), U8.5 (SDA)
- net SCL: now reaches J15.2 (Pin_2)
- net SCL: now also U11.15 (PC2), U8.6 (SCL)
- net 5V_fixed: now reaches J16.1 (Pin_1)
- net 5V_fixed: now also U11.17 (VDD), U3.10 (~{SRCLR}), U3.16 (VCC), U8.8 (VCC), C6.2, C9.1
- net BUCK_1: now reaches J16.10 (Pin_10)
- net BUCK_1: now also U11.25 (PD3)
- net O.S_0: now reaches J16.2 (Pin_2)
- net O.S_0: now also U11.1 (PB3)
- net O.S_1: now reaches J16.3 (Pin_3)
- net O.S_1: now also U11.32 (PA4)
- net O:S_2: now reaches J16.4 (Pin_4)
- net O:S_2: now also U11.31 (PD7)
- net BOOST_3: now reaches J16.5 (Pin_5)
- net BOOST_3: now also U11.30 (PB6)
- net BUCK_3: now reaches J16.6 (Pin_6)
- net BUCK_3: now also U11.29 (PB5)
- net BOOST_2: now reaches J16.7 (Pin_7)
- net BOOST_2: now also U11.28 (PB6)
- net BUCK_2: now reaches J16.8 (Pin_8)
- net BUCK_2: now also U11.27 (PD5)
- net BOOST_1: now reaches J16.9 (Pin_9)
- net BOOST_1: now also U11.26 (PD4)
- net GND: now reaches U8.2 (A1)
- net GND: now also U11.33 (GND), U3.13 (~{OE}), U3.8 (GND), U8.3 (A2), U8.4 (GND), U8.7 (WP), C6.1, C9.2
- net CS: now reaches U11.13 (PC0)
- net CS: now also J10.1 (Pin_1)
- net SCK: now reaches U11.19 (PC5)
- net SCK: now also J10.2 (Pin_2)
- net WARNING_1: now reaches U11.2 (PA5)
- net MOSI: now reaches U11.20 (PC6)
- net MOSI: now also J10.3 (Pin_3)
- net MISO: now reaches U11.21 (PC7)
- net MISO: now also J10.4 (Pin_4)
- net at U11.22 (PB4): now also U3.12 (RCLK)
- net at U11.23 (PD1): now also U3.11 (SRCLK)
- net at U11.24 (PD2): now also U3.14 (SER)
- net CRITICAL_1: now reaches U11.3 (PA6)
- net TC_1: now reaches U11.4 (PA7)
- net WARNING_2: now reaches U11.6 (PA1)
- net CRITICAL_2: now reaches U11.7 (PA2)
- net TC_2: now reaches U11.8 (PD0)
- net O.S_3: now reaches U11.9 (PA3)
- net 5V_CTRL: now reaches U3.1 (QB)
- net 12V_CTRL: now reaches U3.15 (QA)
- net 3.3V_CTRL: now reaches U3.2 (QC)
- net REG1_CTRL: now reaches U3.3 (QD)
- net REG2_CTRL: now reaches U3.4 (QE)
- net REG3_CTRL: now reaches U3.5 (QF)
Other:
- moved on the sheet: U3

Commit message: Schematics UPDATE
Parts:
- removed U8: AT24CS04-SSHM, Package_SO:SOIC-8_3.9x4.9mm_P1.27mm, symbol Memory_EEPROM:AT24CS04-SSHM
- added J17: PROG, Connector_PinHeader_2.54mm:PinHeader_1x02_P2.54mm_Vertical, symbol Connector:Conn_01x02_Pin
- added J23: BOT, Connector_PinHeader_2.54mm:PinHeader_1x04_P2.54mm_Vertical, symbol Connector:Conn_01x04_Pin
- added U8: AT24CS32-SSHM, Package_SO:SOIC-8_3.9x4.9mm_P1.27mm, symbol Memory_EEPROM:AT24CS32-SSHM
Connections:
- net 12V_CTRL: now also U3.5 (QF); no longer U3.15 (QA)
- net 3.3V_CTRL: now also U3.3 (QD); no longer U3.2 (QC)
- net 5V_CTRL: now also U3.4 (QE); no longer U3.1 (QB)
- net 5V_fixed: now also U8.8 (VCC)
- net GND: now also U11.23 (PD1), J17.1 (Pin_1), J17.2 (Pin_2), J23.4 (Pin_4), U8.1 (A0), U8.2 (A1), U8.4 (GND), U8.7 (WP)
- net MOSI: now also U11.18 (PC4), U3.11 (SRCLK)
- net REG1_CTRL: now also U3.2 (QC); no longer U3.3 (QD)
- net REG2_CTRL: now also U3.1 (QB); no longer U3.4 (QE)
- net REG3_CTRL: now also U3.15 (QA); no longer U3.5 (QF)
- net SCL: now also U8.6 (SCL)
- net SDA: now also U8.5 (SDA)
- net at U11.10 (PB0): now also J23.1 (Pin_1)
- net at U11.11 (PB1): now also J23.2 (Pin_2)
- net at U11.12 (PB2): now also J23.3 (Pin_3)
- no-connect marks 0 -> 1

Commit message: Schematics UPDATE
Connections:
- net GND: no longer J17.2 (Pin_2), U11.23 (PD1)
- net MOSI: no longer U11.18 (PC4), U3.11 (SRCLK)
- net at U11.22 (PB4): now also U3.14 (SER); no longer U3.12 (RCLK)
- net at U11.24 (PD2): now also U3.12 (RCLK); no longer U3.14 (SER)
- net CRITICAL_1: no longer names the net of U11.3 (PA6)
- net CRITICAL_2: no longer names the net of U11.7 (PA2)
- net O:S_2 renamed O.S_2
- net TC_1: no longer names the net of U11.4 (PA7)
- net TC_2: no longer names the net of U11.8 (PD0)
- net WARNING_1: no longer names the net of U11.2 (PA5)
- net WARNING_2: no longer names the net of U11.6 (PA1)
- new net: J17.2 (Pin_2), U11.23 (PD1)
- new net: U11.18 (PC4), U3.11 (SRCLK)
- no-connect marks 1 -> 11
Changed lines of the file:
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@@
 (kicad_sch
-	(version 20231120)
+	(version 20250114)
 	(generator "eeschema")
-	(generator_version "8.0")
+	(generator_version "9.0")
 	(paper "A4")
+	(text "LOGS"
+		(exclude_from_sim no)
+		(at 202.438 94.742 0)
+		(effects
+			(font
+				(size 3.81 3.81)
+			)
+		)
+	)
 	(junction
 		(at 189.23 109.22)
@@
 	)
 	(junction
-		(at 153.67 110.49)
-		(diameter 0)
-		(color 0 0 0 0)
-	)
-	(junction
 		(at 125.73 144.78)
 		(diameter 0)
@@
 	)
 	(no_connect
+		(at 104.14 118.11)
+	)
+	(no_connect
+		(at 128.27 137.16)
+	)
+	(no_connect
+		(at 104.14 123.19)
+	)
+	(no_connect
+		(at 104.14 115.57)
+	)
+	(no_connect
+		(at 176.53 71.12)
+	)
+	(no_connect
 		(at 190.5 111.76)
 	)
+	(no_connect
+		(at 104.14 113.03)
+	)
+	(no_connect
+		(at 104.14 125.73)
+	)
+	(no_connect
+		(at 104.14 128.27)
+	)
+	(no_connect
+		(at 104.14 120.65)
+	)
+	(no_connect
+		(at 176.53 68.58)
+	)
 	(wire
 		(pts
@@
 	(wire
 		(pts
+			(xy 137.16 113.03) (xy 137.16 125.73)
+		)
+		(stroke
+			(width 0)
+			(type default)
+		)
+	)
+	(wire
+		(pts
 			(xy 107.95 149.86) (xy 107.95 143.51)
 		)
@@
 	(wire
 		(pts
+			(xy 144.78 53.34) (xy 156.21 53.34)
+		)
+		(stroke
+			(width 0)
+			(type default)
+		)
+	)
+	(wire
+		(pts
 			(xy 125.73 138.43) (xy 158.75 138.43)
 		)
@@
 	(wire
 		(pts
-			(xy 162.56 110.49) (xy 153.67 110.49)
-		)
-		(stroke
-			(width 0)
-			(type default)
-		)
-	)
-	(wire
-		(pts
-			(xy 91.44 123.19) (xy 104.14 123.19)
+			(xy 146.05 109.22) (xy 146.05 111.76)
 		)
 		(stroke
@@
 	(wire
 		(pts
-			(xy 91.44 128.27) (xy 104.14 128.27)
-		)
-		(stroke
-			(width 0)
-			(type default)
-		)
-	)
-	(wire
-		(pts
 			(xy 190.5 106.68) (xy 189.23 106.68)
 		)
@@
 	(wire
 		(pts
-			(xy 134.62 125.73) (xy 138.43 125.73)
+			(xy 134.62 125.73) (xy 137.16 125.73)
 		)
 		(stroke
@@
 	(wire
 		(pts
-			(xy 146.05 110.49) (xy 146.05 111.76)
-		)
-		(stroke
-			(width 0)
-			(type default)
-		)
-	)
-	(wire
-		(pts
 			(xy 118.11 154.94) (xy 118.11 142.24)
 		)
@@
 	(wire
 		(pts
-			(xy 146.05 111.76) (xy 137.16 111.76)
+			(xy 146.05 111.76) (xy 135.89 111.76)
 		)
 		(stroke
@@
 	(wire
 		(pts
-			(xy 91.44 113.03) (xy 104.14 113.03)
+			(xy 142.24 66.04) (xy 156.21 66.04)
 		)
 		(stroke
@@
 	(wire
 		(pts
-			(xy 91.44 125.73) (xy 104.14 125.73)
-		)
-		(stroke
-			(width 0)
-			(type default)
-		)
-	)
-	(wire
-		(pts
-			(xy 138.43 113.03) (xy 138.43 125.73)
-		)
-		(stroke
-			(width 0)
-			(type default)
-		)
-	)
-	(wire
-		(pts
 			(xy 160.02 129.54) (xy 160.02 139.7)
 		)
@@
 	(wire
 		(pts
-			(xy 144.78 115.57) (xy 144.78 66.04)
-		)
-		(stroke
-			(width 0)
-			(type default)
-		)
-	)
-	(wire
-		(pts
 			(xy 189.23 119.38) (xy 200.66 119.38)
 		)
@@
 	(wire
 		(pts
+			(xy 146.05 109.22) (xy 162.56 109.22)
+		)
+		(stroke
+			(width 0)
+			(type default)
+		)
+	)
+	(wire
+		(pts
 			(xy 190.5 109.22) (xy 189.23 109.22)
 		)
@@
 	(wire
 		(pts
-			(xy 144.78 66.04) (xy 156.21 66.04)
-		)
-		(stroke
-			(width 0)
-			(type default)
-		)
-	)
-	(wire
-		(pts
 			(xy 176.53 66.04) (xy 180.34 66.04)
 		)
@@
 	(wire
 		(pts
-			(xy 91.44 115.57) (xy 104.14 115.57)
-		)
-		(stroke
-			(width 0)
-			(type default)
-		)
-	)
-	(wire
-		(pts
 			(xy 120.65 92.71) (xy 120.65 101.6)
 		)
@@
 	(wire
 		(pts
-			(xy 91.44 118.11) (xy 104.14 118.11)
-		)
-		(stroke
-			(width 0)
-			(type default)
-		)
-	)
-	(wire
-		(pts
 			(xy 105.41 139.7) (xy 110.49 139.7)
 		)
@@
 	(wire
 		(pts
-			(xy 143.51 113.03) (xy 138.43 113.03)
+			(xy 143.51 113.03) (xy 137.16 113.03)
 		)
 		(stroke
@@
 	(wire
 		(pts
-			(xy 142.24 53.34) (xy 156.21 53.34)
-		)
-		(stroke
-			(width 0)
-			(type default)
-		)
-	)
-	(wire
-		(pts
 			(xy 115.57 142.24) (xy 115.57 137.16)
 		)
@@
 	(wire
 		(pts
+			(xy 162.56 109.22) (xy 162.56 110.49)
+		)
+		(stroke
+			(width 0)
+			(type default)
+		)
+	)
+	(wire
+		(pts
+			(xy 134.62 123.19) (xy 142.24 123.19)
+		)
+		(stroke
+			(width 0)
+			(type default)
+		)
+	)
+	(wire
+		(pts
 			(xy 134.62 118.11) (xy 142.24 118.11)
 		)
@@
 	(wire
 		(pts
-			(xy 153.67 110.49) (xy 146.05 110.49)
-		)
-		(stroke
-			(width 0)
-			(type default)
-		)
-	)
-	(wire
-		(pts
 			(xy 210.82 111.76) (xy 210.82 119.38)
 		)
@@
 	(wire
 		(pts
-			(xy 142.24 110.49) (xy 142.24 53.34)
-		)
-		(stroke
-			(width 0)
-			(type default)
-		)
-	)
-	(wire
-		(pts
-			(xy 137.16 113.03) (xy 134.62 113.03)
+			(xy 142.24 110.49) (xy 142.24 66.04)
+		)
+		(stroke
+			(width 0)
+			(type default)
+		)
+	)
+	(wire
+		(pts
+			(xy 135.89 113.03) (xy 134.62 113.03)
 		)
 		(stroke
@@
 	(wire
 		(pts
-			(xy 134.62 123.19) (xy 142.24 123.19)
-		)
-		(stroke
-			(width 0)
-			(type default)
-		)
-	)
-	(wire
-		(pts
-			(xy 137.16 111.76) (xy 137.16 113.03)
+			(xy 135.89 111.76) (xy 135.89 113.03)
+		)
+		(stroke
+			(width 0)
+			(type default)
+		)
+	)
+	(wire
+		(pts
+			(xy 144.78 53.34) (xy 144.78 115.57)
 		)
 		(stroke
@@
 			(width 0)
 			(type default)
-		)
-	)
-	(text "LOGS"
-		(exclude_from_sim no)
-		(at 202.438 94.742 0)
-		(effects
-			(font
-				(size 3.81 3.81)
-			)
 		)
 	)
@@
 	)
 	(label "MISO"
-		(at 137.16 118.11 0)
+		(at 138.43 118.11 0)
 		(effects
 			(font
@@
 	)
 	(label "SCK"
-		(at 137.16 123.19 0)
+		(at 139.7 123.19 0)
 		(effects
 			(font
@@
 		)
 	)
-	(label "O:S_2"
+	(label "O.S_2"
 		(at 113.03 100.33 90)
 		(effects
@@
 		)
 	)
-	(hierarchical_label "TC_1"
-		(shape input)
-		(at 91.44 118.11 180)
-		(effects
-			(font
-				(size 1.27 1.27)
-			)
-			(justify right)
-		)
-	)
-	(hierarchical_label "WARNING_1"
-		(shape input)
-		(at 91.44 113.03 180)
-		(effects
-			(font
-				(size 1.27 1.27)
-			)
-			(justify right)
-		)
-	)
 	(hierarchical_label "12V_CTRL"
 		(shape output)
@@
 		)
 	)
-	(hierarchical_label "WARNING_2"
-		(shape input)
-		(at 91.44 123.19 180)
-		(effects
-			(font
-				(size 1.27 1.27)
-			)
-			(justify right)
-		)
-	)
 	(hierarchical_label "REG3_CTRL"
 		(shape output)
@@
 		)
 	)
-	(hierarchical_label "CRITICAL_2"
-		(shape input)
-		(at 91.44 125.73 180)
-		(effects
-			(font
-				(size 1.27 1.27)
-			)
-			(justify right)
-		)
-	)
 	(hierarchical_label "SDA"
 		(shape bidirectional)
@@
 		)
 	)
-	(hierarchical_label "CRITICAL_1"
-		(shape input)
-		(at 91.44 115.57 180)
-		(effects
-			(font
-				(size 1.27 1.27)
-			)
-			(justify right)
-		)
-	)
 	(hierarchical_label "REG2_CTRL"
 		(shape output)
@@
 		)
 	)
-	(hierarchical_label "TC_2"
-		(shape input)
-		(at 91.44 128.27 180)
-		(effects
-			(font
-				(size 1.27 1.27)
-			)
-			(justify right)
-		)
-	)
