File: Tec/HW_Laboratory/Laboratory/control.kicad_sch (KiCad schematic)
At the start: 10 parts, among them J10 SPI, J15 I2C, J16 CONTROL, J17 PROG, J23 BOT, U11 ch32v006k8u6, U3 74HC595, U8 AT24CS32-SSHM

Commit message: Laboratory v2.0:Update the PCB and the Software
Parts:
- added J47: GEN, Connector_PinHeader_2.54mm:PinHeader_1x04_P2.54mm_Vertical, symbol Connector:Conn_01x04_Pin
- added J50: I2C, Connector_PinHeader_2.54mm:PinHeader_1x02_P2.54mm_Vertical, symbol Connector:Conn_01x02_Pin
- added Q7: 2N7002, Package_TO_SOT_SMD:SOT-23, symbol Transistor_FET:2N7002
Connections:
- net 5V_fixed: no longer C6.2, U11.17 (VDD)
- net BOOST_2: now also U11.3 (PA6), J50.2 (Pin_2); no longer J16.7 (Pin_7), U11.28 (PB6)
- net BUCK_2: now also U11.2 (PA5), J50.1 (Pin_1); no longer J16.8 (Pin_8), U11.27 (PD5)
- net GND: now also Q7.2 (S)
- net at U11.5 (PA0): now also J47.1 (Pin_1)
- net at U11.6 (PA1): now also J47.2 (Pin_2)
- net at U11.7 (PA2): now also J47.3 (Pin_3)
- net PWM: now reaches U11.8 (PD0)
- net PWM: now also Q7.1 (G)
- new net: J47.4 (Pin_4), Q7.3 (D)
- new net +3.3V: C6.2, U11.17 (VDD)
- new net Rx: J16.8 (Pin_8), U11.27 (PD5)
- new net Tx: J16.7 (Pin_7), U11.28 (PB6)
- no-connect marks 11 -> 5
Other:
- note added: "Pines Generales"
- note added: "Ventilador"
