File: Tec/HW_Laboratory/Laboratory/iot.kicad_sch (KiCad schematic)
At the start: 2 parts, among them U17 nRF52840

Commit message: Schematics UPDATE
Parts:
- removed AE1: Antenna, RF_Antenna:Texas_SWRA117D_2.4GHz_Right, symbol Device:Antenna
- removed U17: nRF52840, Package_DFN_QFN:Nordic_AQFN-73-1EP_7x7mm_P0.5mm, symbol MCU_Nordic:nRF52840
