File: Tec/HW_Laboratory/Laboratory/Laboratory.kicad_sch (KiCad schematic)
At the start: 0 parts

Commit message: New changes done
Other:
- removed sheet Fuente de alimentacion
- added sheet Fuente_alimentacion (fuente_alimentacion.kicad_sch)
Changed lines of the file:
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@@
 	(paper "A4")
 	(sheet
-		(at 45.72 133.35)
-		(size 52.07 22.86)
+		(at 31.75 20.32)
+		(size 83.82 50.8)
 		(fields_autoplaced yes)
 		(stroke
@@
 			(color 0 0 0 0.0000)
 		)
-		(property "Sheetname" "Fuente de alimentacion"
-			(at 45.72 132.6384 0)
+		(property "Sheetname" "Fuente_alimentacion"
+			(at 31.75 19.6084 0)
 			(effects
 				(font
@@
 			)
 		)
-		(property "Sheetfile" "Alimentacion.kicad_sch"
-			(at 45.72 156.7946 0)
+		(property "Sheetfile" "fuente_alimentacion.kicad_sch"
+			(at 31.75 71.7046 0)
 			(effects
 				(font

Commit message: Schematics UPDATE
Other:
- added sheet Control_central (Control_central.kicad_sch)
- added sheet Generador_funciones (generador_funciones.kicad_sch)
- added sheet IoT (iot.kicad_sch)
Changed lines of the file:
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@@
 	(paper "A4")
+	(sheet
+		(at 31.75 139.7)
+		(size 83.82 53.34)
+		(fields_autoplaced yes)
+		(stroke
+			(width 0.1524)
+			(type solid)
+		)
+		(fill
+			(color 0 0 0 0.0000)
+		)
+		(property "Sheetname" "Control_central"
+			(at 31.75 138.9884 0)
+			(effects
+				(font
+					(size 1.27 1.27)
+				)
+				(justify left bottom)
+			)
+		)
+		(property "Sheetfile" "Control_central.kicad_sch"
+			(at 31.75 193.6246 0)
+			(effects
+				(font
+					(size 1.27 1.27)
+				)
+				(justify left top)
+			)
+		)
+		(instances
+			(project "Laboratory"
+				(path "/91075eda-b6cb-4282-964d-615bb20560a9"
+					(page "8")
+				)
+			)
+		)
+	)
 	(sheet
 		(at 31.75 20.32)
@@
 				)
 			)
+		)
+	)
+	(sheet
+		(at 152.4 20.32)
+		(size 88.9 49.53)
+		(fields_autoplaced yes)
+		(stroke
+			(width 0.1524)
+			(type solid)
+		)
+		(fill
+			(color 0 0 0 0.0000)
+		)
+		(property "Sheetname" "Generador_funciones"
+			(at 152.4 19.6084 0)
+			(effects
+				(font
+					(size 1.27 1.27)
+				)
+				(justify left bottom)
+			)
+		)
+		(property "Sheetfile" "generador_funciones.kicad_sch"
+			(at 152.4 70.4346 0)
+			(effects
+				(font
+					(size 1.27 1.27)
+				)
+				(justify left top)
+			)
+		)
+		(instances
+			(project "Laboratory"
+				(path "/91075eda-b6cb-4282-964d-615bb20560a9"
+					(page "9")
+				)
+			)
+		)
+	)
+	(sheet
+		(at 153.67 110.49)
+		(size 87.63 44.45)
+		(fields_autoplaced yes)
+		(stroke
+			(width 0.1524)
+			(type solid)
+		)
+		(fill
+			(color 0 0 0 0.0000)
+		)
+		(property "Sheetname" "IoT"
+			(at 153.67 109.7784 0)
+			(effects
+				(font
+					(size 1.27 1.27)
+				)
+				(justify left bottom)
+			)
+		)
+		(property "Sheetfile" "iot.kicad_sch"
+			(at 153.67 155.5246 0)
+			(effects
+				(font
+					(size 1.27 1.27)
+				)
+				(justify left top)
+			)
+		)
+		(instances
+			(project "Laboratory"
+				(path "/91075eda-b6cb-4282-964d-615bb20560a9"
+					(page "12")
+				)
+			)

Commit message: Schematics UPDATE
Other:
- sheet Control_central renamed Prueba_ESP-CH
- removed sheet IoT
- added sheet Centro_control (centro_control.kicad_sch)
Changed lines of the file:
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@@
 (kicad_sch
-	(version 20231120)
+	(version 20250114)
 	(generator "eeschema")
-	(generator_version "8.0")
+	(generator_version "9.0")
 	(paper "A4")
 	(sheet
 		(at 31.75 139.7)
 		(size 83.82 53.34)
+		(exclude_from_sim no)
+		(in_bom yes)
+		(on_board yes)
+		(dnp no)
 		(fields_autoplaced yes)
 		(stroke
@@
 			(color 0 0 0 0.0000)
 		)
-		(property "Sheetname" "Control_central"
+		(property "Sheetname" "Prueba_ESP-CH"
 			(at 31.75 138.9884 0)
 			(effects
@@
 		(at 31.75 20.32)
 		(size 83.82 50.8)
+		(exclude_from_sim no)
+		(in_bom yes)
+		(on_board yes)
+		(dnp no)
 		(fields_autoplaced yes)
 		(stroke
@@
 		(at 152.4 20.32)
 		(size 88.9 49.53)
+		(exclude_from_sim no)
+		(in_bom yes)
+		(on_board yes)
+		(dnp no)
 		(fields_autoplaced yes)
 		(stroke
@@
 	)
 	(sheet
-		(at 153.67 110.49)
-		(size 87.63 44.45)
+		(at 166.37 116.84)
+		(size 82.55 41.91)
+		(exclude_from_sim no)
+		(in_bom yes)
+		(on_board yes)
+		(dnp no)
 		(fields_autoplaced yes)
 		(stroke
@@
 			(color 0 0 0 0.0000)
 		)
-		(property "Sheetname" "IoT"
-			(at 153.67 109.7784 0)
+		(property "Sheetname" "Centro_control"
+			(at 166.37 116.1284 0)
 			(effects
 				(font
@@
 			)
 		)
-		(property "Sheetfile" "iot.kicad_sch"
-			(at 153.67 155.5246 0)
+		(property "Sheetfile" "centro_control.kicad_sch"
+			(at 166.37 159.3346 0)
 			(effects
 				(font
@@
 			(project "Laboratory"
 				(path "/91075eda-b6cb-4282-964d-615bb20560a9"
-					(page "12")
+					(page "11")
 				)
 			)
@@
 		)
 	)
+	(embedded_fonts no)
 )

Commit message: Schematics UPDATE
Other:
- sheet Prueba_ESP-CH renamed Analizador
Changed lines of the file:
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@@
 			(color 0 0 0 0.0000)
 		)
-		(property "Sheetname" "Prueba_ESP-CH"
+		(property "Sheetname" "Analizador"
 			(at 31.75 138.9884 0)
 			(effects
