File: Tec/HW_Laboratory/Laboratory/generador_funciones.kicad_sch (KiCad schematic)
At the start: 59 parts, among them J18 AUX, J19 BOT, J20 OUT, J21 Pot3, J22 PROG, J24 I2C, J25 POWER, J26 Pot1, J27 Pot2, J33 Pot6, J34 Pot4, J35 Pot5, U13 LM358, U14 74HC595, U15 CH32V003AxMx, U16 AT24CS32-SSHM, U19 74HC595, U20 LM358, U21 AT24CS32-SSHM

Commit message: Schematics UPDATE
Connections:
- net SDA: now reaches J24.1 (Pin_1), U15.1 (PC1), U16.5 (SDA), U21.5 (SDA)
- net SCL: now reaches J24.2 (Pin_2), U15.2 (PC2), U16.6 (SCL), U21.6 (SCL)
- no-connect marks 6 -> 9
Changed lines of the file:
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@@
+	)
+	(no_connect
+		(at 76.2 101.6)
+	)
+	(no_connect
+		(at 196.85 110.49)
 	)
 	(no_connect
@@
 	)
 	(no_connect
+		(at 92.71 74.93)
+	)
+	(no_connect
 		(at 163.83 29.21)
 	)
@@
 		)
 	)
+	(label "SCL"
+		(at 140.97 115.57 0)
+		(effects
+			(font
+				(size 1.27 1.27)
+			)
+			(justify left bottom)
+		)
+	)
+	(label "SDA"
+		(at 139.7 113.03 0)
+		(effects
+			(font
+				(size 1.27 1.27)
+			)
+			(justify left bottom)
+		)
+	)
