File: Tec/HW_Laboratory/Laboratory/Adaptacion.kicad_sch (KiCad schematic)
At the start: 16 parts, among them Q10 BSS138, Q11 BSS138, Q12 BSS138, Q13 BSS138, Q14 BSS138, Q15 BSS138, Q16 BSS138, Q17 BSS138

Commit message: Digital analizer UPDATE
Parts:
- added Q19, Q21, Q22: BSS138, Package_TO_SOT_SMD:SOT-23, symbol Transistor_FET:BSS138
- added R85, R86, R87: 1k, Resistor_SMD:R_0603_1608Metric, symbol Device:R
Connections:
- net GND6: now also Q19.2 (S), Q21.2 (S), Q22.2 (S)
- net Anal_3.3V: now reaches R73.2
- net Anal_3.3V: now also R16.2, R17.2, R23.2, R24.2, R72.2, R74.2, R75.2, R85.2, R86.2, R87.2
- new net CS_in: Q21.1 (G)
- new net CS_out: Q21.3 (D), R86.1
- new net MISO_in: Q19.1 (G)
- new net MISO_out: Q19.3 (D), R85.1
- new net Rx_in: Q22.1 (G)
- new net Rx_out: Q22.3 (D), R87.1
