File: Tec/HW_Laboratory/Laboratory/Laboratory.kicad_pcb (KiCad board)
At the start: 2 copper layers, 100 x 100 mm, 13 parts, among them J2 Conn_01x08_Pin, J3 Conn_01x08_Pin, Q1 AO3401A, Q2 AO3401A, Q3 AO3401A, Q4 AO3401A, Q5 AO3401A, Q6 AO3401A, U1 74HC595, U2 INA3221

Commit message: New changes done
Parts:
- removed Q3, Q4, Q5, Q6: AO3401A, Package_TO_SOT_SMD:SOT-23
- added ?: , , F.Cu at (176.6, 103.6)
- added ?: , , F.Cu at (117.5, 103.8)
- added C1: 100uF, Capacitor_SMD:C_Elec_5x5.4, F.Cu at (105.5, 128.1)
- added C2: 220uF, Capacitor_SMD:C_Elec_5x5.4, F.Cu at (88.7, 120.6)
- added C3: 22uF, Capacitor_SMD:C_0603_1608Metric, F.Cu at (108.2, 124.3)
- added C4: 22uF, Capacitor_SMD:C_0603_1608Metric, F.Cu at (90.4, 126.1)
- added C5: 100nF, Capacitor_SMD:C_0603_1608Metric, F.Cu at (107.5, 103.8)
- added D1: SS34, Diode_SMD:D_SMA, F.Cu at (97.0, 119.4)
- added D2: SS34, Diode_SMD:D_SMA, F.Cu at (87.3, 127.6)
- added D3: SS34, Diode_SMD:D_SMA, F.Cu at (82.6, 122.1)
- added D4: SS34, Diode_SMD:D_SMA, F.Cu at (82.7, 129.6)
- added D5: BUCK, LED_SMD:LED_0603_1608Metric, F.Cu at (100.5, 109.2)
- added D6: BOOST, LED_SMD:LED_0603_1608Metric, F.Cu at (105.6, 123.5)
- added D7: BZX84Cxx, Package_TO_SOT_SMD:SOT-23, F.Cu at (134.8, 107.7)
- added H1: MountingHole_Pad, MountingHole:MountingHole_2.2mm_M2_DIN965_Pad, F.Cu at (83.0, 89.4)
- added H2: MountingHole_Pad, MountingHole:MountingHole_2.2mm_M2_DIN965_Pad, F.Cu at (111.5, 89.4)
- added H3: MountingHole_Pad, MountingHole:MountingHole_2.2mm_M2_DIN965_Pad, F.Cu at (82.7, 137.5)
- added H4: MountingHole_Pad, MountingHole:MountingHole_2.2mm_M2_DIN965_Pad, F.Cu at (111.2, 137.5)
- added J1: ENTRADA, TerminalBlock_Phoenix:TerminalBlock_Phoenix_PT-1,5-8-3.5-H_1x08_P3.50mm_Horizontal, F.Cu at (120.3, 108.4)
- added J10: SPI, Connector_PinHeader_2.54mm:PinHeader_1x04_P2.54mm_Vertical, F.Cu at (136.2, 137.9)
- added J11: A0, Connector_PinHeader_1.00mm:PinHeader_1x03_P1.00mm_Vertical, F.Cu at (84.5, 93.3)
- added J12: A1, Connector_PinHeader_1.00mm:PinHeader_1x03_P1.00mm_Vertical, F.Cu at (86.5, 93.3)
- added J13: I2C, Connector_PinHeader_2.54mm:PinHeader_1x02_P2.54mm_Vertical, F.Cu at (107.1, 99.4)
- added J14: CON1, Connector_PinHeader_2.54mm:PinHeader_1x02_P2.54mm_Vertical, F.Cu at (104.6, 94.3)
- added J15: I2C, Connector_PinHeader_2.54mm:PinHeader_1x02_P2.54mm_Vertical, F.Cu at (151.6, 138.0)
- added J16: CONTROL, Connector_PinHeader_2.54mm:PinHeader_1x10_P2.54mm_Vertical, F.Cu at (135.1, 103.2)
- added J4: CONTROL, Connector_PinHeader_2.54mm:PinHeader_1x02_P2.54mm_Vertical, F.Cu at (98.2, 138.2)
- added J5: OUT, TerminalBlock_Phoenix:TerminalBlock_Phoenix_PT-1,5-2-3.5-H_1x02_P3.50mm_Horizontal, F.Cu at (87.8, 135.0)
- added J6: A2, Connector_PinHeader_1.00mm:PinHeader_1x03_P1.00mm_Vertical, F.Cu at (92.5, 93.3)
- added J7: A0, Connector_PinHeader_1.00mm:PinHeader_1x03_P1.00mm_Vertical, F.Cu at (106.6, 105.8)
- added J8: A2, Connector_PinHeader_1.00mm:PinHeader_1x03_P1.00mm_Vertical, F.Cu at (110.8, 110.3)
- added J9: A1, Connector_PinHeader_1.00mm:PinHeader_1x03_P1.00mm_Vertical, F.Cu at (110.8, 108.3)
- added L1: 22uH, Inductor_SMD:L_7.3x7.3_H4.5, F.Cu at (96.3, 126.6)
- added L2: 22uH, Inductor_SMD:L_7.3x7.3_H4.5, F.Cu at (107.9, 117.6)
- added R4: 10k, Resistor_SMD:R_0603_1608Metric, F.Cu at (100.5, 112.5)
- added R5: 10k, Resistor_SMD:R_0603_1608Metric, F.Cu at (104.3, 103.8)
- added R6: 10k, Resistor_SMD:R_0603_1608Metric, F.Cu at (103.3, 105.7)
- added R7: 330, Resistor_SMD:R_0603_1608Metric, F.Cu at (99.7, 106.7)
- added R8: 330, Resistor_SMD:R_0603_1608Metric, F.Cu at (104.0, 123.5)
- added R9: 10k, Resistor_SMD:R_0603_1608Metric, F.Cu at (138.6, 108.7)
- added REF**: MountingHole_2.2mm_M2_DIN965_Pad, MountingHole:MountingHole_2.2mm_M2_DIN965_Pad, F.Cu at (176.8, 137.4)
- added REF**: MountingHole_2.2mm_M2_DIN965_Pad, MountingHole:MountingHole_2.2mm_M2_DIN965_Pad, F.Cu at (117.7, 137.6)
- added U10: LM75B, Package_SO:SOIC-8_3.9x4.9mm_P1.27mm, F.Cu at (105.3, 109.7)
- added U11: ch32v006k8u6, Package_DFN_QFN:QFN-32-1EP_4x4mm_P0.4mm_EP2.65x2.65mm, F.Cu at (148.0, 131.2)
- added U3: 74HC595, Package_SO:SOIC-16W_5.3x10.2mm_P1.27mm, F.Cu at (139.0, 129.1)
- added U5: INA3221, Package_DFN_QFN:Texas_RGV0016A_VQFN-16-1EP_4x4mm_P0.65mm_EP2.1x2.1mm, F.Cu at (164.9, 106.0)
- added U6: INA3221, Package_DFN_QFN:Texas_RGV0016A_VQFN-16-1EP_4x4mm_P0.65mm_EP2.1x2.1mm, F.Cu at (164.9, 135.0)
- added U7: LM75B, Package_SO:SOIC-8_3.9x4.9mm_P1.27mm, F.Cu at (154.2, 125.0)
- added U8: AT24CS04-SSHM, Package_SO:SOIC-8_3.9x4.9mm_P1.27mm, F.Cu at (127.9, 137.2)
- added U9: DS1803, Package_DIP:DIP-16_W7.62mm, F.Cu at (100.1, 95.6)
- J2: value Conn_01x08_Pin -> SALIDA; footprint Connector_PinHeader_2.54mm:PinHeader_1x08_P2.54mm_Vertical -> TerminalBlock_Phoenix:TerminalBlock_Phoenix_PT-1,5-8-3.5-H_1x08_P3.50mm_Horizontal
- J3: value Conn_01x08_Pin -> IN; footprint Connector_PinHeader_2.54mm:PinHeader_1x08_P2.54mm_Vertical -> TerminalBlock_Phoenix:TerminalBlock_Phoenix_PT-1,5-2-3.5-H_1x02_P3.50mm_Horizontal
- Q2: value AO3401A -> BC847BS; footprint Package_TO_SOT_SMD:SOT-23 -> Package_TO_SOT_SMD:SOT-363_SC-70-6
- R1: value 0.01 -> 11.5k; footprint Resistor_SMD:R_2512_6332Metric -> Resistor_SMD:R_0603_1608Metric
- R2: value 0.01 -> 5k; footprint Resistor_SMD:R_2512_6332Metric -> Resistor_SMD:R_0603_1608Metric
- R3: value 0.01 -> 95k; footprint Resistor_SMD:R_2512_6332Metric -> Resistor_SMD:R_0603_1608Metric
- U1: value 74HC595 -> LM2596S-ADJ; footprint Package_SO:SOP-16_4.4x10.4mm_P1.27mm -> Package_TO_SOT_SMD:TO-263-5_TabPin3
- U2: value INA3221 -> MT3608; footprint Package_DFN_QFN:Texas_RGV0016A_VQFN-16-1EP_4x4mm_P0.65mm_EP2.1x2.1mm -> Package_TO_SOT_SMD:SOT-23-6
- moved J2 92.1 mm to (174.5, 132.5), turned to 90 degrees
- moved Q2 46.2 mm to (134.9, 120.2), turned to 90 degrees
- moved Q1 42.7 mm to (130.3, 107.7)
- moved J3 29.6 mm to (102.7, 135.0)
- moved R3 29.4 mm to (90.4, 129.7)
- moved R2 23.2 mm to (94.6, 132.5), turned to 90 degrees
- moved U1 18.6 mm to (87.2, 111.0), turned to 180 degrees
- moved U2 17.7 mm to (97.4, 133.1), turned to -90 degrees
- moved R1 15.1 mm to (98.7, 110.3), turned to -90 degrees
Connections:
- J2 pad 1: /Fuente de alimentacion/Consumo/GND -> unconnected-(J2-Pin_1-Pad1)
- J2 pad 2: Net-(J2-Pin_2) -> unconnected-(J2-Pin_2-Pad2)
- J2 pad 3: Net-(J2-Pin_3) -> unconnected-(J2-Pin_3-Pad3)
- J2 pad 4: Net-(J2-Pin_4) -> unconnected-(J2-Pin_4-Pad4)
- J2 pad 5: Net-(J2-Pin_5) -> unconnected-(J2-Pin_5-Pad5)
- J2 pad 6: Net-(J2-Pin_6) -> unconnected-(J2-Pin_6-Pad6)
- J2 pad 7: Net-(J2-Pin_7) -> unconnected-(J2-Pin_7-Pad7)
- J2 pad 8: /Fuente de alimentacion/Consumo/GND -> unconnected-(J2-Pin_8-Pad8)
- J3 pad 1: /Fuente de alimentacion/Consumo/GND -> /Fuente_alimentacion/Regulador/Vin
- J3 pad 2: unconnected-(J3-Pin_2-Pad2) -> GND1
- Q1 pad 1: Net-(Q1-G) -> unconnected-(Q1-G-Pad1)
- Q1 pad 2: Net-(J2-Pin_2) -> unconnected-(Q1-S-Pad2)
- Q1 pad 3: /Fuente de alimentacion/Consumo/3.3V -> unconnected-(Q1-D-Pad3)
- Q2 pad 1: Net-(Q2-G) -> unconnected-(Q2A-E1-Pad1)
- Q2 pad 2: Net-(J2-Pin_3) -> unconnected-(Q2A-B1-Pad2)
- Q2 pad 3: /Fuente de alimentacion/Consumo/5V -> unconnected-(Q2B-C2-Pad3)
- R1 pad 1: Net-(J3-Pin_7) -> /Fuente_alimentacion/Regulador/FB_BUCK
- R1 pad 2: /Fuente de alimentacion/Consumo/3.3V -> GND1
- R2 pad 1: Net-(U2-IN+2) -> GND1
- R2 pad 2: /Fuente de alimentacion/Consumo/5V -> /Fuente_alimentacion/Regulador/FB_BOOST
- R3 pad 1: Net-(J3-Pin_5) -> Net-(U9-W1)
- R3 pad 2: /Fuente de alimentacion/Consumo/12V -> /Fuente_alimentacion/Regulador/FB_BOOST
- U1 pad 1: Net-(Q2-G) -> /Fuente_alimentacion/Regulador/Vin
- U1 pad 2: Net-(Q3-G) -> /Fuente_alimentacion/Regulador/OUT_BUCK
- U1 pad 3: Net-(Q4-G) -> GND1
- U1 pad 4: Net-(Q5-G) -> /Fuente_alimentacion/Regulador/FB_BUCK
- U1 pad 5: Net-(Q6-G) -> /Fuente_alimentacion/Regulador/BUCK
- U2 pad 1: /Fuente de alimentacion/Consumo/3.3V -> /Fuente_alimentacion/Regulador/SW_BOOST
- U2 pad 2: Net-(J3-Pin_7) -> GND1
- U2 pad 3: /Fuente de alimentacion/Consumo/GND -> /Fuente_alimentacion/Regulador/FB_BOOST
- U2 pad 4: unconnected-(U2-VS-Pad4) -> /Fuente_alimentacion/Regulador/BOOST
- U2 pad 5: /Fuente de alimentacion/Consumo/GND -> /Fuente_alimentacion/Regulador/Vin
Routing:
- net GND1: track 0.00 -> 155.6 mm, vias 0 -> 1
- net /Fuente_alimentacion/Regulador/5V: track 0.00 -> 75.7 mm, vias 0 -> 4
- net /Fuente_alimentacion/Regulador/Vout_boost: track 0.00 -> 57.8 mm, vias 0 -> 2
- net /Fuente_alimentacion/Regulador/Vin: track 0.00 -> 44.7 mm
- net /Fuente_alimentacion/Regulador/Vout_buck: track 0.00 -> 42.1 mm, vias 0 -> 2
- net Net-(U9-W1): track 0.00 -> 40.1 mm, vias 0 -> 4
- net /Fuente_alimentacion/Regulador/BUCK: track 0.00 -> 39.6 mm, vias 0 -> 1
- net /Fuente_alimentacion/Regulador/SW_BOOST: track 0.00 -> 37.9 mm, vias 0 -> 2
- net SCL: track 0.00 -> 34.0 mm, vias 0 -> 1
- net SDA: track 0.00 -> 32.2 mm, vias 0 -> 2
- net Net-(J14-Pin_1): track 0.00 -> 30.0 mm, vias 0 -> 2
- net /Fuente_alimentacion/Regulador/OUT_BUCK: track 0.00 -> 21.2 mm
- net /Fuente_alimentacion/Regulador/FB_BUCK: track 0.00 -> 18.2 mm
- net /Fuente_alimentacion/Regulador/BOOST: track 0.00 -> 18.1 mm
- net Net-(Q1-G): track 15.2 -> 0.00 mm
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- added copper zone on F.Cu, net /Fuente_alimentacion/Regulador/OUT_BUCK
- added copper zone on F.Cu, net /Fuente_alimentacion/Regulador/SW_BOOST
- added copper zone on F.Cu, net /Fuente_alimentacion/Regulador/Vin
- added copper zone on F.Cu, net /Fuente_alimentacion/Regulador/Vout_buck
- added copper zone on B.Cu, net GND1
- added copper zone on F.Cu, net GND1
Other:
- board size 100 x 100 mm -> 99.3 x 99.6 mm
- board text added: "12V"
- board text added: "5V"
- board text added: "BOOST"
- board text added: "BUCK"
- board text added: "GND"
- board text added: "O.S"
- board text added: "OPC"
- board text added: "Power supply buck-boost lm2596/mt3608 Luis Miguel Carmona Cortés"
- board text added: "SCL"
- board text added: "SDA"
- board text added: "VCC"

Commit message: Schematics UPDATE
Parts:
- added C10: 100nF, Capacitor_SMD:C_0603_1608Metric, F.Cu at (135.7, 134.9)
- added C6: 100nF, Capacitor_SMD:C_0603_1608Metric, F.Cu at (152.3, 133.8)
- added C7: 100nF, Capacitor_SMD:C_0603_1608Metric, F.Cu at (158.8, 135.2)
- added C8: 100nF, Capacitor_SMD:C_0603_1608Metric, F.Cu at (166.4, 106.1)
- added C9: 100nF, Capacitor_SMD:C_0603_1608Metric, F.Cu at (141.9, 128.1)
- added D10: BZX84Cxx, Package_TO_SOT_SMD:SOT-23, F.Cu at (137.2, 117.2)
- added D11: BZX84Cxx, Package_TO_SOT_SMD:SOT-23, F.Cu at (141.8, 117.2)
- added D12: BZX84Cxx, Package_TO_SOT_SMD:SOT-23, F.Cu at (146.4, 117.2)
- added D8: BZX84Cxx, Package_TO_SOT_SMD:SOT-23, F.Cu at (127.9, 117.2)
- added D9: BZX84Cxx, Package_TO_SOT_SMD:SOT-23, F.Cu at (132.5, 117.2)
- added Q3: AO3401A, Package_TO_SOT_SMD:SOT-23, F.Cu at (127.9, 112.3)
- added Q4: BC847BS, Package_TO_SOT_SMD:SOT-363_SC-70-6, F.Cu at (140.1, 107.7)
- added Q5: AO3401A, Package_TO_SOT_SMD:SOT-23, F.Cu at (132.5, 112.3)
- added Q6: AO3401A, Package_TO_SOT_SMD:SOT-23, F.Cu at (137.2, 112.3)
- added Q7: BC847BS, Package_TO_SOT_SMD:SOT-363_SC-70-6, F.Cu at (144.0, 107.7)
- added Q8: AO3401A, Package_TO_SOT_SMD:SOT-23, F.Cu at (141.8, 112.3)
- added Q9: AO3401A, Package_TO_SOT_SMD:SOT-23, F.Cu at (146.4, 112.3)
- added R10: 10k, Resistor_SMD:R_0603_1608Metric, F.Cu at (126.8, 107.8)
- added R11: 10k, Resistor_SMD:R_0603_1608Metric, F.Cu at (129.3, 107.8)
- added R12: 10k, Resistor_SMD:R_0603_1608Metric, F.Cu at (131.8, 107.8)
- added R13: 10k, Resistor_SMD:R_0603_1608Metric, F.Cu at (134.3, 107.8)
- added R14: 10k, Resistor_SMD:R_0603_1608Metric, F.Cu at (136.8, 107.8)
- added R15: 10k, Resistor_SMD:R_0603_1608Metric, F.Cu at (164.4, 133.8)
- added R16: 10k, Resistor_SMD:R_0603_1608Metric, F.Cu at (164.3, 135.9)
- added R17: 10k, Resistor_SMD:R_0603_1608Metric, F.Cu at (161.2, 135.9)
- added R18: 10k, Resistor_SMD:R_0603_1608Metric, F.Cu at (161.2, 133.8)
- added R19: 10k, Resistor_SMD:R_0603_1608Metric, F.Cu at (164.4, 102.6)
- added R20: 10k, Resistor_SMD:R_0603_1608Metric, F.Cu at (166.4, 104.5)
- added R21: 10k, Resistor_SMD:R_0603_1608Metric, F.Cu at (163.3, 104.2)
- added R22: 10k, Resistor_SMD:R_0603_1608Metric, F.Cu at (160.2, 103.0)
- added R23: 10k, Resistor_SMD:R_0603_1608Metric, F.Cu at (160.9, 105.4)
- added R24: 10k, Resistor_SMD:R_0603_1608Metric, F.Cu at (163.3, 106.2)
- added R25: 10k, Resistor_SMD:R_0603_1608Metric, F.Cu at (164.2, 137.5)
- added R26: 10k, Resistor_SMD:R_0603_1608Metric, F.Cu at (161.2, 137.5)
- added R27: 10k, Resistor_SMD:R_0603_1608Metric, F.Cu at (136.5, 129.0)
- added R28: 10k, Resistor_SMD:R_0603_1608Metric, F.Cu at (134.9, 131.2)
- added R29: 10k, Resistor_SMD:R_0603_1608Metric, F.Cu at (136.5, 132.2)
- added R30: 10m, Resistor_SMD:R_2512_6332Metric, F.Cu at (168.3, 129.8)
- added R31: 10m, Resistor_SMD:R_2512_6332Metric, F.Cu at (157.5, 129.8)
- added R32: 10m, Resistor_SMD:R_2512_6332Metric, F.Cu at (163.0, 123.5)
- added R33: 10m, Resistor_SMD:R_2512_6332Metric, F.Cu at (157.8, 110.7)
- added R34: 10m, Resistor_SMD:R_2512_6332Metric, F.Cu at (163.2, 116.9)
- added R35: 10m, Resistor_SMD:R_2512_6332Metric, F.Cu at (168.3, 110.8)
- moved R9 28.4 mm to (126.3, 134.3)
- moved U6 24.8 mm to (163.2, 110.3), turned to 180 degrees
- moved D7 24.4 mm to (130.9, 131.8)
- moved Q1 24.4 mm to (126.8, 131.8)
- moved U5 24.2 mm to (163.1, 130.2)
- moved U8 17.3 mm to (139.6, 124.5)
- moved U7 15.1 mm to (141.1, 132.6)
- moved U3 11.0 mm to (149.2, 124.8)
- moved Q2 10.6 mm to (128.1, 128.3)
- moved J16 5.50 mm to (129.6, 103.3)
- moved J15 3.40 mm to (148.2, 137.9)
- moved U11 1.49 mm to (148.1, 132.6)
Connections:
- D7 pad 1: unconnected-(D7-A-Pad1) -> Net-(D7-A)
- D7 pad 3: unconnected-(D7-K-Pad3) -> /Fuente_alimentacion/Selector/12V_IN
- J1 pad 1: unconnected-(J1-Pin_1-Pad1) -> GND2
- J1 pad 2: unconnected-(J1-Pin_2-Pad2) -> /Fuente_alimentacion/Selector/5V_fixed
- J1 pad 3: unconnected-(J1-Pin_3-Pad3) -> /Fuente_alimentacion/Selector/REG3_IN
- J1 pad 4: unconnected-(J1-Pin_4-Pad4) -> /Fuente_alimentacion/Selector/REG2_IN
- J1 pad 5: unconnected-(J1-Pin_5-Pad5) -> /Fuente_alimentacion/Selector/REG1_IN
- J1 pad 6: unconnected-(J1-Pin_6-Pad6) -> /Fuente_alimentacion/Selector/3.3V_IN
- J1 pad 7: unconnected-(J1-Pin_7-Pad7) -> /Fuente_alimentacion/Selector/5V_IN
- J1 pad 8: unconnected-(J1-Pin_8-Pad8) -> /Fuente_alimentacion/Selector/12V_IN
- J10 pad 1: unconnected-(J10-Pin_1-Pad1) -> /Fuente_alimentacion/Selector/Control/CS
- J10 pad 2: unconnected-(J10-Pin_2-Pad2) -> /Fuente_alimentacion/Selector/Control/SCK
- J10 pad 3: unconnected-(J10-Pin_3-Pad3) -> /Fuente_alimentacion/Selector/Control/MOSI
- J10 pad 4: unconnected-(J10-Pin_4-Pad4) -> /Fuente_alimentacion/Selector/Control/MISO
- J15 pad 1: unconnected-(J15-Pin_1-Pad1) -> /Fuente_alimentacion/Selector/SDA
- J15 pad 2: unconnected-(J15-Pin_2-Pad2) -> /Fuente_alimentacion/Selector/SCL
- J16 pad 1: unconnected-(J16-Pin_1-Pad1) -> /Fuente_alimentacion/Selector/5V_fixed
- J16 pad 10: unconnected-(J16-Pin_10-Pad10) -> /Fuente_alimentacion/Selector/Control/BUCK_1
- J16 pad 2: unconnected-(J16-Pin_2-Pad2) -> /Fuente_alimentacion/Selector/Control/O.S_0
- J16 pad 3: unconnected-(J16-Pin_3-Pad3) -> /Fuente_alimentacion/Selector/Control/O.S_1
- J16 pad 4: unconnected-(J16-Pin_4-Pad4) -> /Fuente_alimentacion/Selector/Control/O:S_2
- J16 pad 5: unconnected-(J16-Pin_5-Pad5) -> /Fuente_alimentacion/Selector/Control/BOOST_3
- J16 pad 6: unconnected-(J16-Pin_6-Pad6) -> /Fuente_alimentacion/Selector/Control/BUCK_3
- J16 pad 7: unconnected-(J16-Pin_7-Pad7) -> /Fuente_alimentacion/Selector/Control/BOOST_2
- J16 pad 8: unconnected-(J16-Pin_8-Pad8) -> /Fuente_alimentacion/Selector/Control/BUCK_2
- J16 pad 9: unconnected-(J16-Pin_9-Pad9) -> /Fuente_alimentacion/Selector/Control/BOOST_1
- J2 pad 1: unconnected-(J2-Pin_1-Pad1) -> /Fuente_alimentacion/Selector/12V_OUT
- J2 pad 2: unconnected-(J2-Pin_2-Pad2) -> /Fuente_alimentacion/Selector/5V_OUT
- J2 pad 3: unconnected-(J2-Pin_3-Pad3) -> /Fuente_alimentacion/Selector/3.3V_OUT
- J2 pad 4: unconnected-(J2-Pin_4-Pad4) -> /Fuente_alimentacion/Selector/REG1_OUT
- J2 pad 5: unconnected-(J2-Pin_5-Pad5) -> /Fuente_alimentacion/Selector/REG2_OUT
- J2 pad 6: unconnected-(J2-Pin_6-Pad6) -> /Fuente_alimentacion/Selector/REG3_OUT
- J2 pad 7: unconnected-(J2-Pin_7-Pad7) -> /Fuente_alimentacion/Selector/5V_fixed
- J2 pad 8: unconnected-(J2-Pin_8-Pad8) -> GND2
- Q1 pad 1: unconnected-(Q1-G-Pad1) -> Net-(D7-A)
- Q1 pad 2: unconnected-(Q1-S-Pad2) -> /Fuente_alimentacion/Selector/Mosfets/12V_OUT
- Q1 pad 3: unconnected-(Q1-D-Pad3) -> /Fuente_alimentacion/Selector/12V_IN
- Q2 pad 1: unconnected-(Q2A-E1-Pad1) -> GND2
- Q2 pad 2: unconnected-(Q2A-B1-Pad2) -> /Fuente_alimentacion/Selector/Control/12V_CTRL
- Q2 pad 3: unconnected-(Q2B-C2-Pad3) -> Net-(D8-A)
- Q2 pad 4: unconnected-(Q2B-E2-Pad4) -> GND2
- Q2 pad 5: unconnected-(Q2B-B2-Pad5) -> /Fuente_alimentacion/Selector/Control/5V_CTRL
- Q2 pad 6: unconnected-(Q2A-C1-Pad6) -> Net-(D7-A)
- R9 pad 1: unconnected-(R9-Pad1) -> Net-(D7-A)
- R9 pad 2: unconnected-(R9-Pad2) -> /Fuente_alimentacion/Selector/12V_IN
- U11 pad 1: unconnected-(U11-PB3-Pad1) -> /Fuente_alimentacion/Selector/Control/O.S_0
- U11 pad 13: unconnected-(U11-PC0-Pad13) -> /Fuente_alimentacion/Selector/Control/CS
- U11 pad 14: unconnected-(U11-PC1-Pad14) -> /Fuente_alimentacion/Selector/SDA
- U11 pad 15: unconnected-(U11-PC2-Pad15) -> /Fuente_alimentacion/Selector/SCL
- U11 pad 17: unconnected-(U11-VDD-Pad17) -> /Fuente_alimentacion/Selector/5V_fixed
- U11 pad 19: unconnected-(U11-PC5-Pad19) -> /Fuente_alimentacion/Selector/Control/SCK
- U11 pad 2: unconnected-(U11-PA5-Pad2) -> /Fuente_alimentacion/Selector/Control/WARNING_1
- U11 pad 20: unconnected-(U11-PC6-Pad20) -> /Fuente_alimentacion/Selector/Control/MOSI
- U11 pad 21: unconnected-(U11-PC7-Pad21) -> /Fuente_alimentacion/Selector/Control/MISO
- U11 pad 22: unconnected-(U11-PB4-Pad22) -> Net-(U11-PB4)
- U11 pad 23: unconnected-(U11-PD1-Pad23) -> Net-(U11-PD1)
- U11 pad 24: unconnected-(U11-PD2-Pad24) -> Net-(U11-PD2)
- U11 pad 25: unconnected-(U11-PD3-Pad25) -> /Fuente_alimentacion/Selector/Control/BUCK_1
- U11 pad 26: unconnected-(U11-PD4-Pad26) -> /Fuente_alimentacion/Selector/Control/BOOST_1
- U11 pad 27: unconnected-(U11-PD5-Pad27) -> /Fuente_alimentacion/Selector/Control/BUCK_2
- U11 pad 28: unconnected-(U11-PB6-Pad28) -> /Fuente_alimentacion/Selector/Control/BOOST_2
- U11 pad 29: unconnected-(U11-PB5-Pad29) -> /Fuente_alimentacion/Selector/Control/BUCK_3
- U11 pad 3: unconnected-(U11-PA6-Pad3) -> /Fuente_alimentacion/Selector/Control/CRITICAL_1
- U11 pad 30: unconnected-(U11-PB6-Pad30) -> /Fuente_alimentacion/Selector/Control/BOOST_3
- U11 pad 31: unconnected-(U11-PD7-Pad31) -> /Fuente_alimentacion/Selector/Control/O:S_2
- U11 pad 32: unconnected-(U11-PA4-Pad32) -> /Fuente_alimentacion/Selector/Control/O.S_1
- U11 pad 33: unconnected-(U11-GND-Pad33) -> GND2
- U11 pad 4: unconnected-(U11-PA7-Pad4) -> /Fuente_alimentacion/Selector/Control/TC_1
- U11 pad 6: unconnected-(U11-PA1-Pad6) -> /Fuente_alimentacion/Selector/Control/WARNING_2
- U11 pad 7: unconnected-(U11-PA2-Pad7) -> /Fuente_alimentacion/Selector/Control/CRITICAL_2
- U11 pad 8: unconnected-(U11-PD0-Pad8) -> /Fuente_alimentacion/Selector/Control/TC_2
- U11 pad 9: unconnected-(U11-PA3-Pad9) -> /Fuente_alimentacion/Selector/Control/O.S_3
- U3 pad 1: unconnected-(U3-QB-Pad1) -> /Fuente_alimentacion/Selector/Control/5V_CTRL
- U3 pad 10: unconnected-(U3-~{SRCLR}-Pad10) -> /Fuente_alimentacion/Selector/5V_fixed
- U3 pad 11: unconnected-(U3-SRCLK-Pad11) -> Net-(U11-PD1)
- U3 pad 12: unconnected-(U3-RCLK-Pad12) -> Net-(U11-PB4)
- U3 pad 13: unconnected-(U3-~{OE}-Pad13) -> GND2
- U3 pad 14: unconnected-(U3-SER-Pad14) -> Net-(U11-PD2)
- U3 pad 15: unconnected-(U3-QA-Pad15) -> /Fuente_alimentacion/Selector/Control/12V_CTRL
- U3 pad 16: unconnected-(U3-VCC-Pad16) -> /Fuente_alimentacion/Selector/5V_fixed
- U3 pad 2: unconnected-(U3-QC-Pad2) -> /Fuente_alimentacion/Selector/Control/3.3V_CTRL
- U3 pad 3: unconnected-(U3-QD-Pad3) -> /Fuente_alimentacion/Selector/Control/REG1_CTRL
- U3 pad 4: unconnected-(U3-QE-Pad4) -> /Fuente_alimentacion/Selector/Control/REG2_CTRL
- U3 pad 5: unconnected-(U3-QF-Pad5) -> /Fuente_alimentacion/Selector/Control/REG3_CTRL
- U3 pad 8: unconnected-(U3-GND-Pad8) -> GND2
- U5 pad 1: unconnected-(U5-IN-3-Pad1) -> /Fuente_alimentacion/Selector/3.3V_OUT
- U5 pad 10: unconnected-(U5-PV-Pad10) -> Net-(U5-PV)
- U5 pad 11: unconnected-(U5-IN-1-Pad11) -> /Fuente_alimentacion/Selector/12V_OUT
- U5 pad 12: unconnected-(U5-IN+1-Pad12) -> /Fuente_alimentacion/Selector/Mosfets/12V_OUT
- U5 pad 13: unconnected-(U5-TC-Pad13) -> /Fuente_alimentacion/Selector/Control/TC_1
- U5 pad 14: unconnected-(U5-IN-2-Pad14) -> /Fuente_alimentacion/Selector/5V_OUT
- U5 pad 15: unconnected-(U5-IN+2-Pad15) -> /Fuente_alimentacion/Selector/Mosfets/5V_OUT
- U5 pad 16: unconnected-(U5-VPU-Pad16) -> Net-(U5-VPU)
- U5 pad 17: unconnected-(U5-EP-Pad17) -> GND2
- U5 pad 2: unconnected-(U5-IN+3-Pad2) -> /Fuente_alimentacion/Selector/Mosfets/3.3V_OUT
- U5 pad 3: unconnected-(U5-GND-Pad3) -> GND2
- U5 pad 4: unconnected-(U5-VS-Pad4) -> /Fuente_alimentacion/Selector/5V_fixed
- U5 pad 5: unconnected-(U5-A0-Pad5) -> GND2
- U5 pad 6: unconnected-(U5-SCL-Pad6) -> /Fuente_alimentacion/Selector/SCL
- U5 pad 7: unconnected-(U5-SDA-Pad7) -> /Fuente_alimentacion/Selector/SDA
- U5 pad 8: unconnected-(U5-WARNING-Pad8) -> /Fuente_alimentacion/Selector/Control/WARNING_1
- U5 pad 9: unconnected-(U5-CRITICAL-Pad9) -> /Fuente_alimentacion/Selector/Control/CRITICAL_1
- U6 pad 1: unconnected-(U6-IN-3-Pad1) -> /Fuente_alimentacion/Selector/REG3_OUT
- U6 pad 10: unconnected-(U6-PV-Pad10) -> Net-(U6-PV)
- U6 pad 11: unconnected-(U6-IN-1-Pad11) -> /Fuente_alimentacion/Selector/REG1_OUT
- U6 pad 12: unconnected-(U6-IN+1-Pad12) -> /Fuente_alimentacion/Selector/Mosfets/REG1_OUT
- U6 pad 13: unconnected-(U6-TC-Pad13) -> /Fuente_alimentacion/Selector/Control/TC_2
- U6 pad 14: unconnected-(U6-IN-2-Pad14) -> /Fuente_alimentacion/Selector/REG2_OUT
- U6 pad 15: unconnected-(U6-IN+2-Pad15) -> /Fuente_alimentacion/Selector/Mosfets/REG2_OUT
- U6 pad 16: unconnected-(U6-VPU-Pad16) -> Net-(U6-VPU)
- U6 pad 17: unconnected-(U6-EP-Pad17) -> GND2
- U6 pad 2: unconnected-(U6-IN+3-Pad2) -> /Fuente_alimentacion/Selector/Mosfets/REG3_OUT
- U6 pad 3: unconnected-(U6-GND-Pad3) -> GND2
- U6 pad 4: unconnected-(U6-VS-Pad4) -> /Fuente_alimentacion/Selector/5V_fixed
- U6 pad 5: unconnected-(U6-A0-Pad5) -> /Fuente_alimentacion/Selector/5V_fixed
- U6 pad 6: unconnected-(U6-SCL-Pad6) -> /Fuente_alimentacion/Selector/SCL
- U6 pad 7: unconnected-(U6-SDA-Pad7) -> /Fuente_alimentacion/Selector/SDA
- U6 pad 8: unconnected-(U6-WARNING-Pad8) -> /Fuente_alimentacion/Selector/Control/WARNING_2
- U6 pad 9: unconnected-(U6-CRITICAL-Pad9) -> /Fuente_alimentacion/Selector/Control/CRITICAL_2
- U7 pad 1: unconnected-(U7-SDA-Pad1) -> /Fuente_alimentacion/Selector/SDA
- U7 pad 2: unconnected-(U7-SCL-Pad2) -> /Fuente_alimentacion/Selector/SCL
- U7 pad 3: unconnected-(U7-O.S.-Pad3) -> /Fuente_alimentacion/Selector/Control/O.S_3
- U7 pad 4: unconnected-(U7-GND-Pad4) -> GND2
- U7 pad 5: unconnected-(U7-A2-Pad5) -> GND2
- U7 pad 6: unconnected-(U7-A1-Pad6) -> GND2
- U7 pad 7: unconnected-(U7-A0-Pad7) -> GND2
- U7 pad 8: unconnected-(U7-+Vs-Pad8) -> /Fuente_alimentacion/Selector/5V_fixed
- U8 pad 2: unconnected-(U8-A1-Pad2) -> GND2
- U8 pad 3: unconnected-(U8-A2-Pad3) -> GND2
- U8 pad 4: unconnected-(U8-GND-Pad4) -> GND2
- U8 pad 5: unconnected-(U8-SDA-Pad5) -> /Fuente_alimentacion/Selector/SDA
- U8 pad 6: unconnected-(U8-SCL-Pad6) -> /Fuente_alimentacion/Selector/SCL
- U8 pad 7: unconnected-(U8-WP-Pad7) -> GND2
- U8 pad 8: unconnected-(U8-VCC-Pad8) -> /Fuente_alimentacion/Selector/5V_fixed

Commit message: Schematics UPDATE
Parts:
- added AE1: Antenna, RF_Antenna:Texas_SWRA117D_2.4GHz_Right, F.Cu at (121.1, 53.0)
- added D13: WS2812B, LED_SMD:LED_WS2812B_PLCC4_5.0x5.0mm_P3.2mm, F.Cu at (84.3, 44.2)
- added H5: MountingHole_Pad, MountingHole:MountingHole_2.2mm_M2_DIN965_Pad, F.Cu at (117.9, 97.2)
- added H6: MountingHole_Pad, MountingHole:MountingHole_2.2mm_M2_DIN965_Pad, F.Cu at (176.6, 97.2)
- added H7: MountingHole_Pad, MountingHole:MountingHole_2.2mm_M2_DIN965_Pad, F.Cu at (117.9, 72.7)
- added H8: MountingHole_Pad, MountingHole:MountingHole_2.2mm_M2_DIN965_Pad, F.Cu at (176.7, 72.8)
- added J17: PROG, Connector_PinHeader_2.54mm:PinHeader_1x02_P2.54mm_Vertical, F.Cu at (168.5, 138.0)
- added J18: AUX, Connector_PinHeader_2.54mm:PinHeader_1x02_P2.54mm_Vertical, F.Cu at (150.7, 72.0)
- added J19: BOT, Connector_PinHeader_2.54mm:PinHeader_1x04_P2.54mm_Vertical, F.Cu at (139.8, 97.7)
- added J20: OUT, Connector_PinHeader_2.54mm:PinHeader_1x03_P2.54mm_Vertical, F.Cu at (141.3, 72.0)
- added J21: Pot3, Connector_PinHeader_2.54mm:PinHeader_1x03_P2.54mm_Vertical, F.Cu at (122.3, 97.7)
- added J22: PROG, Connector_PinHeader_2.54mm:PinHeader_1x02_P2.54mm_Vertical, F.Cu at (151.5, 97.8)
- added J23: BOT, Connector_PinHeader_2.54mm:PinHeader_1x04_P2.54mm_Vertical, F.Cu at (141.6, 138.2)
- added J24: I2C, Connector_PinHeader_2.54mm:PinHeader_1x02_P2.54mm_Vertical, F.Cu at (159.0, 97.8)
- added J25: POWER, Connector_PinHeader_2.54mm:PinHeader_1x02_P2.54mm_Vertical, F.Cu at (144.3, 97.7)
- added J26: Pot1, Connector_PinHeader_2.54mm:PinHeader_1x03_P2.54mm_Vertical, F.Cu at (118.1, 87.3)
- added J27: Pot2, Connector_PinHeader_2.54mm:PinHeader_1x03_P2.54mm_Vertical, F.Cu at (118.2, 77.4)
- added J28: Conn_01x04_Pin, Connector_PinHeader_2.54mm:PinHeader_1x04_P2.54mm_Vertical, F.Cu at (111.1, 52.9)
- added J29: Conn_01x08_Pin, Connector_PinHeader_2.54mm:PinHeader_1x08_P2.54mm_Vertical, F.Cu at (111.5, 78.8)
- added J30: Conn_01x08_Pin, Connector_PinHeader_2.54mm:PinHeader_1x08_P2.54mm_Vertical, F.Cu at (88.9, 82.8)
- added J31: Conn_01x08_Pin, Connector_PinHeader_2.54mm:PinHeader_1x08_P2.54mm_Vertical, F.Cu at (82.8, 61.5)
- added J32: Conn_01x08_Pin, Connector_PinHeader_2.54mm:PinHeader_1x08_P2.54mm_Vertical, F.Cu at (105.5, 68.6)
- added J33: Pot6, Connector_PinHeader_2.54mm:PinHeader_1x03_P2.54mm_Vertical, F.Cu at (166.4, 97.8)
- added J34: Pot4, Connector_PinHeader_2.54mm:PinHeader_1x03_P2.54mm_Vertical, F.Cu at (176.6, 87.1)
- added J35: Pot5, Connector_PinHeader_2.54mm:PinHeader_1x03_P2.54mm_Vertical, F.Cu at (176.6, 77.6)
- added R36: 20k, Resistor_SMD:R_0603_1608Metric, F.Cu at (134.5, 80.6)
- added R37: 20k, Resistor_SMD:R_0603_1608Metric, F.Cu at (132.8, 82.1)
- added R38: 10k, Resistor_SMD:R_0603_1608Metric, F.Cu at (132.0, 79.8)
- added R39: 20k, Resistor_SMD:R_0603_1608Metric, F.Cu at (131.3, 82.1)
- added R40: 10k, Resistor_SMD:R_0603_1608Metric, F.Cu at (130.2, 78.4)
- added R41: 20k, Resistor_SMD:R_0603_1608Metric, F.Cu at (129.8, 82.1)
- added R42: 10k, Resistor_SMD:R_0603_1608Metric, F.Cu at (129.1, 79.8)
- added R43: 20k, Resistor_SMD:R_0603_1608Metric, F.Cu at (128.4, 82.1)
- added R44: 10k, Resistor_SMD:R_0603_1608Metric, F.Cu at (127.3, 78.4)
- added R45: 20k, Resistor_SMD:R_0603_1608Metric, F.Cu at (126.9, 82.1)
- added R46: 10k, Resistor_SMD:R_0603_1608Metric, F.Cu at (126.1, 79.8)
- added R47: 20k, Resistor_SMD:R_0603_1608Metric, F.Cu at (125.5, 82.1)
- added R48: 10k, Resistor_SMD:R_0603_1608Metric, F.Cu at (124.3, 78.4)
- added R49: 20k, Resistor_SMD:R_0603_1608Metric, F.Cu at (124.0, 82.1)
- added R50: 10k, Resistor_SMD:R_0603_1608Metric, F.Cu at (123.1, 79.8)
- added R51: 20k, Resistor_SMD:R_0603_1608Metric, F.Cu at (122.5, 82.1)
- added R52: 10k, Resistor_SMD:R_0603_1608Metric, F.Cu at (123.0, 76.2)
- added R53: 10k, Resistor_SMD:R_0603_1608Metric, F.Cu at (132.3, 76.1)
- added R54: 20k, Resistor_SMD:R_0603_1608Metric, F.Cu at (172.7, 77.2)
- added R55: 20k, Resistor_SMD:R_0603_1608Metric, F.Cu at (172.7, 81.7)
- added R56: 10k, Resistor_SMD:R_0603_1608Metric, F.Cu at (172.0, 79.5)
- added R57: 20k, Resistor_SMD:R_0603_1608Metric, F.Cu at (171.2, 81.7)
- added R58: 10k, Resistor_SMD:R_0603_1608Metric, F.Cu at (170.4, 78.0)
- added R59: 20k, Resistor_SMD:R_0603_1608Metric, F.Cu at (169.8, 81.7)
- added R60: 10k, Resistor_SMD:R_0603_1608Metric, F.Cu at (169.0, 79.5)
- added R61: 20k, Resistor_SMD:R_0603_1608Metric, F.Cu at (168.3, 81.7)
- added R62: 10k, Resistor_SMD:R_0603_1608Metric, F.Cu at (167.4, 78.0)
- added R63: 20k, Resistor_SMD:R_0603_1608Metric, F.Cu at (166.9, 81.7)
- added R64: 10k, Resistor_SMD:R_0603_1608Metric, F.Cu at (166.1, 79.5)
- added R65: 20k, Resistor_SMD:R_0603_1608Metric, F.Cu at (165.4, 81.7)
- added R66: 10k, Resistor_SMD:R_0603_1608Metric, F.Cu at (164.5, 78.0)
- added R67: 20k, Resistor_SMD:R_0603_1608Metric, F.Cu at (163.9, 81.7)
- added R68: 10k, Resistor_SMD:R_0603_1608Metric, F.Cu at (163.1, 79.5)
- added R69: 20k, Resistor_SMD:R_0603_1608Metric, F.Cu at (162.5, 81.7)
- added R70: 10k, Resistor_SMD:R_0603_1608Metric, F.Cu at (161.5, 78.0)
- added R71: 10k, Resistor_SMD:R_0603_1608Metric, F.Cu at (158.6, 74.6)
- added U12: ch32v006k8u6, Package_DFN_QFN:QFN-32-1EP_4x4mm_P0.4mm_EP2.65x2.65mm, F.Cu at (98.6, 75.4)
- added U13: LM358, Package_DIP:DIP-8_W7.62mm_Socket, F.Cu at (138.4, 77.8)
- added U14: 74HC595, Package_SO:SOIC-16W_5.3x10.2mm_P1.27mm, F.Cu at (127.6, 88.8)
- added U15: CH32V003AxMx, Package_SO:SOP-16_3.9x9.9mm_P1.27mm, F.Cu at (148.3, 91.7)
- added U16: AT24CS32-SSHM, Package_SO:SOIC-8_3.9x4.9mm_P1.27mm, F.Cu at (137.6, 92.3)
- added U17: nRF52840, Package_DFN_QFN:Nordic_AQFN-73-1EP_7x7mm_P0.5mm, F.Cu at (128.4, 48.5)
- added U18: AT24CS32-SSHM, Package_SO:SOIC-8_3.9x4.9mm_P1.27mm, F.Cu at (84.3, 54.9)
- added U19: 74HC595, Package_SO:SOIC-16W_5.3x10.2mm_P1.27mm, F.Cu at (168.7, 88.5)
- added U20: LM358, Package_DIP:DIP-8_W7.62mm_Socket, F.Cu at (150.3, 77.8)
- added U21: AT24CS32-SSHM, Package_SO:SOIC-8_3.9x4.9mm_P1.27mm, F.Cu at (158.8, 92.1)
- added U4: ESP-12F, RF_Module:ESP-12E, F.Cu at (97.4, 52.8)
- U8: value AT24CS04-SSHM -> AT24CS32-SSHM
- moved R10 25.1 mm to (131.4, 132.5)
- moved Q9 20.4 mm to (126.4, 108.5), turned to 180 degrees
- moved Q4 18.5 mm to (128.6, 122.2)
- moved U7 18.4 mm to (155.1, 120.7)
- moved R28 18.4 mm to (148.9, 119.3)
- moved R27 18.4 mm to (150.5, 117.2)
- moved R29 18.4 mm to (150.5, 120.4)
- moved D12 18.3 mm to (130.3, 108.5), turned to 180 degrees
- moved C10 18.2 mm to (149.7, 123.2)
- moved J10 17.2 mm to (153.4, 138.1), turned to 180 degrees
- moved Q3 16.8 mm to (126.4, 129.0), turned to 180 degrees
- moved Q7 15.9 mm to (128.6, 111.9)
- moved Q8 15.7 mm to (126.4, 115.3), turned to 180 degrees
- moved R11 14.9 mm to (125.2, 122.2), turned to -90 degrees
- moved Q5 14.6 mm to (126.4, 125.5), turned to 180 degrees
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Connections:
- U11 pad 10: unconnected-(U11-PB0-Pad10) -> Net-(J23-Pin_1)
- U11 pad 11: unconnected-(U11-PB1-Pad11) -> Net-(J23-Pin_2)
- U11 pad 12: unconnected-(U11-PB2-Pad12) -> Net-(J23-Pin_3)
- U11 pad 18: unconnected-(U11-PC4-Pad18) -> Net-(U11-PC4)
- U11 pad 23: Net-(U11-PD1) -> GND2
- U3 pad 1: /Fuente_alimentacion/Selector/Control/5V_CTRL -> /Fuente_alimentacion/Selector/Control/REG2_CTRL
- U3 pad 11: Net-(U11-PD1) -> Net-(U11-PC4)
- U3 pad 15: /Fuente_alimentacion/Selector/Control/12V_CTRL -> /Fuente_alimentacion/Selector/Control/REG3_CTRL
- U3 pad 2: /Fuente_alimentacion/Selector/Control/3.3V_CTRL -> /Fuente_alimentacion/Selector/Control/REG1_CTRL
- U3 pad 3: /Fuente_alimentacion/Selector/Control/REG1_CTRL -> /Fuente_alimentacion/Selector/Control/3.3V_CTRL
- U3 pad 4: /Fuente_alimentacion/Selector/Control/REG2_CTRL -> /Fuente_alimentacion/Selector/Control/5V_CTRL
- U3 pad 5: /Fuente_alimentacion/Selector/Control/REG3_CTRL -> /Fuente_alimentacion/Selector/Control/12V_CTRL
- U8 pad 1: unconnected-(U8-NC-Pad1) -> GND2
- U8 pad 3: GND2 -> unconnected-(U8-A2-Pad3)
Routing:
- net /Fuente_alimentacion/Selector/5V_fixed: track 0.00 -> 81.6 mm
- net GND2: track 0.00 -> 53.4 mm
- net /Fuente_alimentacion/Selector/3.3V_OUT: track 0.00 -> 27.6 mm
- net /Fuente_alimentacion/Selector/REG2_OUT: track 0.00 -> 21.0 mm
- net /Fuente_alimentacion/Selector/REG3_IN: track 0.00 -> 16.7 mm
- net /Fuente_alimentacion/Selector/5V_OUT: track 0.00 -> 16.7 mm
- net /Fuente_alimentacion/Selector/REG1_IN: track 0.00 -> 13.8 mm
- net /Fuente_alimentacion/Selector/12V_IN: track 0.00 -> 13.3 mm
- net /Fuente_alimentacion/Selector/REG2_IN: track 0.00 -> 13.2 mm
- net /Fuente_alimentacion/Selector/5V_IN: track 0.00 -> 12.9 mm
- net Net-(D12-A): track 0.00 -> 12.8 mm
- net Net-(D8-A): track 0.00 -> 11.9 mm
- net /Fuente_alimentacion/Selector/3.3V_IN: track 0.00 -> 11.9 mm
- net /Fuente_alimentacion/Selector/REG3_OUT: track 0.00 -> 11.0 mm
- net /Fuente_alimentacion/Selector/12V_OUT: track 0.00 -> 10.9 mm
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Other:
- board text added: "2 DACs r2r of 8 bit each ch32v003/74hc595 Luis Miguel Carmona Cortés"
- board text added: "3.3V"
- board text added: "5V_fixed"
- board text added: "REG1"
- board text added: "REG2"
- board text added: "REG3"

Commit message: Schematics UPDATE
Parts:
- moved J29 4.10 mm to (111.7, 82.9)
- moved J31 3.72 mm to (82.3, 65.1)
Routing:
- net Net-(J31-Pin_1): track 0.00 -> 19.6 mm
- net Net-(J31-Pin_2): track 0.00 -> 17.5 mm
- net Net-(J31-Pin_8): track 0.00 -> 16.8 mm
- net Net-(J31-Pin_3): track 0.00 -> 16.2 mm
- net Net-(J31-Pin_7): track 0.00 -> 16.0 mm
- net Net-(J31-Pin_4): track 0.00 -> 15.4 mm
- net Net-(J31-Pin_6): track 0.00 -> 15.1 mm
- net Net-(J29-Pin_8): track 0.00 -> 14.9 mm
- net Net-(J31-Pin_5): track 0.00 -> 14.5 mm
- net Net-(J29-Pin_7): track 0.00 -> 14.0 mm
- net Net-(J29-Pin_1): track 0.00 -> 13.7 mm
- net Net-(J29-Pin_6): track 0.00 -> 13.1 mm
- net Net-(J32-Pin_8): track 0.00 -> 12.9 mm
- net Net-(J29-Pin_2): track 0.00 -> 12.8 mm
- net Net-(J29-Pin_5): track 0.00 -> 12.2 mm
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