File: Tec/HW_Laboratory/Laboratory/Laboratory.kicad_pcb (KiCad board)
At the start: 2 copper layers, 99.3 x 99.6 mm, 174 parts, among them J1 ENTRADA, J10 SPI, J11 A0, J12 A1, J13 I2C, J14 CON1, J15 I2C, J16 CONTROL, J17 PROG, J18 AUX, J19 BOT, J2 SALIDA, J20 OUT, J21 Pot3, J22 PROG, J23 BOT, J24 I2C, J25 POWER, J26 Pot1, J27 Pot2, J28 Conn_01x04_Pin, J29 Conn_01x08_Pin, J3 IN, J30 Conn_01x08_Pin, J31 Conn_01x08_Pin, J32 Conn_01x08_Pin, J33 Pot6, J34 Pot4, J35 Pot5, J4 CONTROL, J5 OUT, J6 A2, J7 A0, J8 A2, J9 A1, Q1 AO3401A, Q2 BC847BS, Q3 AO3401A, Q4 BC847BS, Q5 AO3401A, Q6 AO3401A, Q7 BC847BS, Q8 AO3401A, Q9 AO3401A, U1 LM2596S-ADJ, U10 LM75B, U11 ch32v006k8u6, U12 ch32v006k8u6, U13 LM358, U14 74HC595, U15 CH32V003AxMx, U16 AT24CS32-SSHM, U17 nRF52840, U18 AT24CS32-SSHM, U19 74HC595, U2 MT3608, U20 LM358, U21 AT24CS32-SSHM, U3 74HC595, U4 ESP-12F, U5 INA3221, U6 INA3221, U7 LM75B, U8 AT24CS32-SSHM, U9 DS1803

Commit message: Schematics UPDATE
Parts:
- removed ? (x2): , 
- removed AE1: Antenna, RF_Antenna:Texas_SWRA117D_2.4GHz_Right
- removed R16, R17, R23, R24: 10k, Resistor_SMD:R_0603_1608Metric
- removed REF** (x2): MountingHole_2.2mm_M2_DIN965_Pad, MountingHole:MountingHole_2.2mm_M2_DIN965_Pad
- added C11: 100nF, Capacitor_SMD:C_0603_1608Metric, F.Cu at (177.3, 59.0)
- added C12: 100nF, Capacitor_SMD:C_0603_1608Metric, F.Cu at (167.5, 59.1)
- added C13: 100nF, Capacitor_SMD:C_0603_1608Metric, F.Cu at (133.4, 49.7)
- added C14: 100nF, Capacitor_SMD:C_0603_1608Metric, F.Cu at (123.1, 49.5)
- added H10: MountingHole_Pad, MountingHole:MountingHole_2.2mm_M2_DIN965_Pad, F.Cu at (176.8, 137.4)
- added H11: MountingHole_Pad, MountingHole:MountingHole_2.2mm_M2_DIN965_Pad, F.Cu at (117.5, 103.8)
- added H12: MountingHole_Pad, MountingHole:MountingHole_2.2mm_M2_DIN965_Pad, F.Cu at (117.7, 137.6)
- added H13: MountingHole_Pad, MountingHole:MountingHole_2.2mm_M2_DIN965_Pad, F.Cu at (176.6, 66.0)
- added H14: MountingHole_Pad, MountingHole:MountingHole_2.2mm_M2_DIN965_Pad, F.Cu at (118.9, 66.0)
- added H15: MountingHole_Pad, MountingHole:MountingHole_2.2mm_M2_DIN965_Pad, F.Cu at (119.0, 43.4)
- added H16: MountingHole_Pad, MountingHole:MountingHole_2.2mm_M2_DIN965_Pad, F.Cu at (176.5, 43.3)
- added H9: MountingHole_Pad, MountingHole:MountingHole_2.2mm_M2_DIN965_Pad, F.Cu at (176.6, 103.6)
- added J36: SPI, Connector_PinHeader_2.54mm:PinHeader_1x04_P2.54mm_Vertical, F.Cu at (138.0, 66.4)
- added J37: USB, Connector_PinHeader_2.54mm:PinHeader_1x04_P2.54mm_Vertical, F.Cu at (124.3, 66.3)
- added J38: IN, TerminalBlock_Phoenix:TerminalBlock_Phoenix_PT-1,5-2-3.5-H_1x02_P3.50mm_Horizontal, F.Cu at (174.5, 51.8)
- added J39: USB_C_Receptacle_USB2.0_16P, Connector_USB:USB_C_Receptacle_GCT_USB4105-xx-A_16P_TopMnt_Horizontal, F.Cu at (118.7, 57.6)
- added SW1: SW_Push, Button_Switch_THT:SW_PUSH_6mm, F.Cu at (129.6, 47.0)
- added SW2: SW_Push, Button_Switch_THT:SW_PUSH_6mm, F.Cu at (133.3, 42.5)
- added U22: AMS1117-3.3, Package_TO_SOT_SMD:SOT-223-3_TabPin2, F.Cu at (109.2, 57.8)
- added U24: AMS1117-3.3, Package_TO_SOT_SMD:SOT-223-3_TabPin2, F.Cu at (172.2, 59.0)
- D13: value WS2812B -> LED; footprint LED_SMD:LED_WS2812B_PLCC4_5.0x5.0mm_P3.2mm -> LED_SMD:LED_0603_1608Metric
- U17: value nRF52840 -> ESP32-S3-WROOM-1; footprint Package_DFN_QFN:Nordic_AQFN-73-1EP_7x7mm_P0.5mm -> RF_Module:ESP32-S3-WROOM-1
- moved D13 90.2 mm to (172.1, 64.8)
- moved R18 87.0 mm to (139.9, 49.5)
- moved R22 61.5 mm to (129.6, 49.7)
- moved U17 24.4 mm to (152.8, 47.0), turned to 0 degrees
- moved U18 7.85 mm to (83.1, 47.1), turned to 90 degrees
- moved J28 2.80 mm to (110.9, 50.1)
- moved J17 2.65 mm to (171.1, 138.0), turned to -90 degrees
- moved U4 1.62 mm to (95.8, 52.8)
- moved R15 0.17 mm to (164.5, 133.8)
Connections:
- net /Fuente_alimentacion/Selector/Control/O:S_2 renamed /Fuente_alimentacion/Selector/Control/O.S_2
- D13 pad 1: unconnected-(D13-VDD-Pad1) -> GND5
- D13 pad 2: unconnected-(D13-DOUT-Pad2) -> Net-(D13-A)
- J17 pad 2: GND2 -> Net-(J17-Pin_2)
- J28 pad 1: unconnected-(J28-Pin_1-Pad1) -> GND3
- R18 pad 1: /Fuente_alimentacion/Selector/Control/TC_1 -> EN
- R18 pad 2: /Fuente_alimentacion/Selector/5V_fixed -> Net-(D13-A)
- R22 pad 1: /Fuente_alimentacion/Selector/Control/CRITICAL_2 -> PROG
- R22 pad 2: /Fuente_alimentacion/Selector/5V_fixed -> Net-(D13-A)
- U11 pad 2: /Fuente_alimentacion/Selector/Control/WARNING_1 -> unconnected-(U11-PA5-Pad2)
- U11 pad 23: GND2 -> Net-(J17-Pin_2)
- U11 pad 3: /Fuente_alimentacion/Selector/Control/CRITICAL_1 -> unconnected-(U11-PA6-Pad3)
- U11 pad 4: /Fuente_alimentacion/Selector/Control/TC_1 -> unconnected-(U11-PA7-Pad4)
- U11 pad 6: /Fuente_alimentacion/Selector/Control/WARNING_2 -> unconnected-(U11-PA1-Pad6)
- U11 pad 7: /Fuente_alimentacion/Selector/Control/CRITICAL_2 -> unconnected-(U11-PA2-Pad7)
- U11 pad 8: /Fuente_alimentacion/Selector/Control/TC_2 -> unconnected-(U11-PD0-Pad8)
- U12 pad 33: unconnected-(U12-GND-Pad33) -> GND3
- U18 pad 8: unconnected-(U18-VCC-Pad8) -> Net-(J29-Pin_1)
- U3 pad 12: Net-(U11-PB4) -> Net-(U11-PD2)
- U3 pad 14: Net-(U11-PD2) -> Net-(U11-PB4)
- U4 pad 10: unconnected-(U4-MISO-Pad10) -> Net-(J29-Pin_5)
- U4 pad 13: unconnected-(U4-MOSI-Pad13) -> Net-(J29-Pin_4)
- U4 pad 14: unconnected-(U4-SCLK-Pad14) -> Net-(J29-Pin_3)
- U5 pad 13: /Fuente_alimentacion/Selector/Control/TC_1 -> unconnected-(U5-TC-Pad13)
- U5 pad 8: /Fuente_alimentacion/Selector/Control/WARNING_1 -> unconnected-(U5-WARNING-Pad8)
- U5 pad 9: /Fuente_alimentacion/Selector/Control/CRITICAL_1 -> unconnected-(U5-CRITICAL-Pad9)
- U6 pad 13: /Fuente_alimentacion/Selector/Control/TC_2 -> unconnected-(U6-TC-Pad13)
- U6 pad 8: /Fuente_alimentacion/Selector/Control/WARNING_2 -> unconnected-(U6-WARNING-Pad8)
- U6 pad 9: /Fuente_alimentacion/Selector/Control/CRITICAL_2 -> unconnected-(U6-CRITICAL-Pad9)
Routing:
- net GND2: track 53.4 -> 308.8 mm, vias 0 -> 18
- net /Fuente_alimentacion/Selector/SCL: track 0.00 -> 97.9 mm, vias 0 -> 13
- net /Fuente_alimentacion/Selector/5V_fixed: track 81.6 -> 179.0 mm, vias 0 -> 3
- net /Fuente_alimentacion/Selector/SDA: track 2.47 -> 92.1 mm, vias 0 -> 7
- net /Fuente_alimentacion/Selector/Mosfets/12V_OUT: track 4.26 -> 61.5 mm, vias 0 -> 4
- net /Fuente_alimentacion/Selector/Mosfets/3.3V_OUT: track 4.98 -> 56.8 mm, vias 0 -> 5
- net /Fuente_alimentacion/Selector/Mosfets/5V_OUT: track 5.96 -> 56.9 mm, vias 0 -> 4
- net /Fuente_alimentacion/Selector/Mosfets/REG3_OUT: track 4.86 -> 55.2 mm, vias 0 -> 2
- net /Fuente_alimentacion/Selector/Mosfets/REG2_OUT: track 5.80 -> 47.6 mm, vias 0 -> 4
- net /Fuente_alimentacion/Selector/Control/O.S_3: track 2.20 -> 37.6 mm, vias 0 -> 4
- net /Fuente_alimentacion/Selector/Mosfets/REG1_OUT: track 4.52 -> 36.7 mm, vias 0 -> 4
- net /Fuente_alimentacion/Selector/Control/O.S_0: track 0.00 -> 31.5 mm, vias 0 -> 1
- net /Fuente_alimentacion/Selector/Control/O.S_1: track 0.00 -> 30.5 mm, vias 0 -> 1
- net /Fuente_alimentacion/Selector/REG1_OUT: track 5.46 -> 35.2 mm
- net /Fuente_alimentacion/Selector/Control/BUCK_1: track 0.00 -> 29.3 mm, vias 0 -> 1
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- added copper zone on B.Cu, net GND2
- added copper zone on F.Cu, net GND2
Other:
- board text added: "BOOST_1"
- board text added: "BOOST_2"
- board text added: "BOST_3"
- board text added: "BOTON_1"
- board text added: "BOTON_2"
- board text added: "BOTON_3"
- board text added: "BUCK_1"
- board text added: "BUCK_2"
- board text added: "BUCK_3"
- board text added: "CS"
- board text added: "DNM"
- board text added: "MISO"
- board text added: "MOSI"
- board text added: "O.S_0"
- board text added: "O.S_1"
- board text added: "O.S_2"
- board text added: "SCK"
- board text added: "SWI"

Commit message: Schematics UPDATE
Parts:
- removed J30, J31, J32: Conn_01x08_Pin, Connector_PinHeader_2.54mm:PinHeader_1x08_P2.54mm_Vertical
- removed U17: ESP32-S3-WROOM-1, RF_Module:ESP32-S3-WROOM-1
- removed U18: AT24CS32-SSHM, Package_SO:SOIC-8_3.9x4.9mm_P1.27mm
- added C15: 100nF, Capacitor_SMD:C_0603_1608Metric, F.Cu at (90.0, 61.1)
- added C16: 100nF, Capacitor_SMD:C_0603_1608Metric, F.Cu at (90.0, 64.2)
- added C17: 100nF, Capacitor_SMD:C_0603_1608Metric, F.Cu at (142.0, 49.6)
- added D14: LED, LED_SMD:LED_0603_1608Metric, F.Cu at (92.2, 63.1)
- added H17: MountingHole_Pad, MountingHole:MountingHole_2.2mm_M2_DIN965_Pad, F.Cu at (111.2, 43.3)
- added H18: MountingHole_Pad, MountingHole:MountingHole_2.2mm_M2_DIN965_Pad, F.Cu at (82.8, 43.3)
- added H19: MountingHole_Pad, MountingHole:MountingHole_2.2mm_M2_DIN965_Pad, F.Cu at (111.5, 81.9)
- added H20: MountingHole_Pad, MountingHole:MountingHole_2.2mm_M2_DIN965_Pad, F.Cu at (83.1, 81.9)
- added J40: POWER, TerminalBlock_Phoenix:TerminalBlock_Phoenix_PT-1,5-2-3.5-H_1x02_P3.50mm_Horizontal, F.Cu at (109.4, 62.4)
- added J41: SPI, Connector_PinHeader_2.54mm:PinHeader_1x04_P2.54mm_Vertical, F.Cu at (94.3, 83.1)
- added J42: UART, Connector_PinHeader_2.54mm:PinHeader_1x02_P2.54mm_Vertical, F.Cu at (87.1, 83.2)
- added Q10: BSS138, Package_TO_SOT_SMD:SOT-23, F.Cu at (84.1, 50.0)
- added Q11: BSS138, Package_TO_SOT_SMD:SOT-23, F.Cu at (87.8, 50.0)
- added Q12: BSS138, Package_TO_SOT_SMD:SOT-23, F.Cu at (91.5, 50.0)
- added Q13: BSS138, Package_TO_SOT_SMD:SOT-23, F.Cu at (95.1, 50.0)
- added Q14: BSS138, Package_TO_SOT_SMD:SOT-23, F.Cu at (109.8, 50.1)
- added Q15: BSS138, Package_TO_SOT_SMD:SOT-23, F.Cu at (98.8, 50.1)
- added Q16: BSS138, Package_TO_SOT_SMD:SOT-23, F.Cu at (102.5, 50.1)
- added Q17: BSS138, Package_TO_SOT_SMD:SOT-23, F.Cu at (106.1, 50.1)
- added Q18: BC547, Package_TO_SOT_THT:TO-92_Inline, F.Cu at (157.3, 53.5)
- added Q20: BC547, Package_TO_SOT_THT:TO-92_Inline, F.Cu at (151.6, 53.5)
- added R16: 1k, Resistor_SMD:R_0603_1608Metric, F.Cu at (84.1, 53.7)
- added R17: 1k, Resistor_SMD:R_0603_1608Metric, F.Cu at (87.8, 53.7)
- added R23: 1k, Resistor_SMD:R_0603_1608Metric, F.Cu at (91.5, 53.7)
- added R24: 1k, Resistor_SMD:R_0603_1608Metric, F.Cu at (95.1, 53.7)
- added R72: 1k, Resistor_SMD:R_0603_1608Metric, F.Cu at (109.7, 53.7)
- added R73: 1k, Resistor_SMD:R_0603_1608Metric, F.Cu at (98.8, 53.7)
- added R74: 1k, Resistor_SMD:R_0603_1608Metric, F.Cu at (102.5, 53.7)
- added R75: 1k, Resistor_SMD:R_0603_1608Metric, F.Cu at (106.1, 53.7)
- added R76: 10k, Resistor_SMD:R_0603_1608Metric, F.Cu at (160.6, 61.0)
- added R77: 10k, Resistor_SMD:R_0603_1608Metric, F.Cu at (172.6, 42.5)
- added R78: 10k, Resistor_SMD:R_0603_1608Metric, F.Cu at (160.6, 64.0)
- added R79: 10k, Resistor_SMD:R_0603_1608Metric, F.Cu at (153.1, 58.9)
- added R80: 10k, Resistor_SMD:R_0603_1608Metric, F.Cu at (153.1, 57.1)
- added U23: ESP-12F, RF_Module:ESP-12E, F.Cu at (174.7, 54.9)
- added U25: CH340C, Package_SO:SOIC-16_3.9x9.9mm_P1.27mm, F.Cu at (140.4, 55.4)
- J28: value Conn_01x04_Pin -> USB_C_Receptacle_USB2.0_16P; footprint Connector_PinHeader_2.54mm:PinHeader_1x04_P2.54mm_Vertical -> Connector_USB:USB_C_Receptacle_GCT_USB4105-xx-A_16P_TopMnt_Horizontal
- J29: value Conn_01x08_Pin -> Analizador; footprint Connector_PinHeader_2.54mm:PinHeader_1x08_P2.54mm_Vertical -> Connector_PinHeader_2.54mm:PinHeader_2x04_P2.54mm_Vertical
- J37: value USB -> UART
- U12: value ch32v006k8u6 -> W25Q128JVS; footprint Package_DFN_QFN:QFN-32-1EP_4x4mm_P0.4mm_EP2.65x2.65mm -> Package_SO:SOIC-8_5.3x5.3mm_P1.27mm
- U4: value ESP-12F -> RP2040; footprint RF_Module:ESP-12E -> Package_DFN_QFN:QFN-56-1EP_7x7mm_P0.4mm_EP3.2x3.2mm
- moved J38 55.0 mm to (119.6, 56.0), turned to -90 degrees
- moved C11 43.6 mm to (133.7, 57.6)
- moved C12 43.6 mm to (124.0, 57.6)
- moved D13 43.6 mm to (128.5, 63.4)
- moved U24 43.6 mm to (128.6, 57.5)
- moved J29 41.2 mm to (94.1, 45.6), turned to 90 degrees
- moved J37 39.3 mm to (163.6, 67.2)
- moved J28 36.0 mm to (83.9, 73.9), turned to -90 degrees
- moved U22 25.0 mm to (84.8, 62.9), turned to 180 degrees
- moved U4 20.5 mm to (96.2, 73.3)
- moved R22 18.9 mm to (148.5, 49.0)
- moved SW2 18.9 mm to (152.2, 42.0)
- moved R18 18.9 mm to (158.7, 49.0)
- moved SW1 17.8 mm to (147.4, 46.5)
- moved C13 17.3 mm to (149.8, 44.2), turned to 90 degrees
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Connections:
- net Net-(J24-Pin_1) renamed /Generador_funciones/SDA
- net Net-(J24-Pin_2) renamed /Generador_funciones/SCL
- net Net-(U17-USB_D+) renamed /Centro_control/TTL-USB/UD+
- net Net-(U17-USB_D-) renamed /Centro_control/TTL-USB/UD-
- C12 pad 1: Net-(J38-Pin_2) -> /Centro_control/TTL-USB/VUSB
- J29 pad 1: Net-(J29-Pin_1) -> unconnected-(J29-Pin_1-Pad1)
- J29 pad 2: Net-(J29-Pin_2) -> unconnected-(J29-Pin_2-Pad2)
- J29 pad 3: Net-(J29-Pin_3) -> unconnected-(J29-Pin_3-Pad3)
- J29 pad 4: Net-(J29-Pin_4) -> unconnected-(J29-Pin_4-Pad4)
- J29 pad 5: Net-(J29-Pin_5) -> unconnected-(J29-Pin_5-Pad5)
- J29 pad 6: Net-(J29-Pin_6) -> unconnected-(J29-Pin_6-Pad6)
- J29 pad 7: Net-(J29-Pin_7) -> unconnected-(J29-Pin_7-Pad7)
- J29 pad 8: Net-(J29-Pin_8) -> unconnected-(J29-Pin_8-Pad8)
- J37 pad 2: Net-(J37-Pin_2) -> /Centro_control/TTL-USB/Tx
- J37 pad 3: Net-(J37-Pin_3) -> /Centro_control/TTL-USB/Rx
- J38 pad 1: GND5 -> /Centro_control/TTL-USB/VUSB
- J38 pad 2: Net-(J38-Pin_2) -> GND5
- J39 pad A4: Net-(J38-Pin_2) -> /Centro_control/TTL-USB/VUSB
- J39 pad A9: Net-(J38-Pin_2) -> /Centro_control/TTL-USB/VUSB
- J39 pad B4: Net-(J38-Pin_2) -> /Centro_control/TTL-USB/VUSB
- J39 pad B9: Net-(J38-Pin_2) -> /Centro_control/TTL-USB/VUSB
- U12 pad 1: Net-(J31-Pin_1) -> unconnected-(U12-~{CS}-Pad1)
- U12 pad 2: Net-(J31-Pin_2) -> unconnected-(U12-DO/IO_{1}-Pad2)
- U12 pad 3: Net-(J31-Pin_3) -> unconnected-(U12-~{WP}/IO_{2}-Pad3)
- U12 pad 4: Net-(J31-Pin_4) -> unconnected-(U12-GND-Pad4)
- U12 pad 5: Net-(J31-Pin_5) -> unconnected-(U12-DI/IO_{0}-Pad5)
- U12 pad 6: Net-(J31-Pin_6) -> unconnected-(U12-CLK-Pad6)
- U12 pad 7: Net-(J31-Pin_7) -> unconnected-(U12-~{HOLD}/~{RESET}/IO_{3}-Pad7)
- U12 pad 8: Net-(J31-Pin_8) -> unconnected-(U12-VCC-Pad8)
- U22 pad 1: GND3 -> GND6
- U22 pad 2: Net-(J28-Pin_4) -> Net-(D14-A)
- U22 pad 3: Net-(J29-Pin_1) -> Net-(J40-Pin_2)
- U24 pad 2: Net-(J38-Pin_2) -> /Centro_control/TTL-USB/VUSB
- U4 pad 1: unconnected-(U4-~{RST}-Pad1) -> Net-(U4-IOVDD-Pad1)
- U4 pad 10: Net-(J29-Pin_5) -> Net-(U4-IOVDD-Pad1)
- U4 pad 13: Net-(J29-Pin_4) -> unconnected-(U4-GPIO10-Pad13)
- U4 pad 14: Net-(J29-Pin_3) -> unconnected-(U4-GPIO11-Pad14)
- U4 pad 15: GND3 -> unconnected-(U4-GPIO12-Pad15)
- U4 pad 21: Net-(J28-Pin_2) -> unconnected-(U4-XOUT-Pad21)
- U4 pad 22: Net-(J28-Pin_3) -> Net-(U4-IOVDD-Pad1)
- U4 pad 8: Net-(J28-Pin_4) -> unconnected-(U4-GPIO6-Pad8)
Routing:
- net GND4: track 15.6 -> 269.3 mm, vias 0 -> 1
- net GND5: track 0.00 -> 168.9 mm
- net 5V_gen: track 0.00 -> 86.9 mm, vias 0 -> 7
- net Net-(U14-SER): track 0.00 -> 50.4 mm, vias 0 -> 4
- net Net-(U14-SRCLK): track 0.00 -> 49.4 mm, vias 0 -> 4
- net Net-(U14-RCLK): track 0.00 -> 49.1 mm, vias 0 -> 2
- net Net-(J20-Pin_1): track 0.00 -> 39.0 mm
- net Net-(D13-A): track 0.00 -> 37.2 mm
- net Net-(J29-Pin_1): track 37.2 -> 0.00 mm
- net /Generador_funciones/SCL: track 0.00 -> 36.2 mm
- net Net-(J20-Pin_3): track 0.00 -> 33.8 mm
- net /Centro_control/TTL-USB/VUSB: track 0.00 -> 33.0 mm
- net Net-(J34-Pin_3): track 18.5 -> 50.1 mm
- net Net-(J26-Pin_3): track 15.7 -> 46.7 mm
- net /Generador_funciones/SDA: track 0.00 -> 30.5 mm
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- added copper zone on B.Cu, net GND4
- added copper zone on F.Cu, net GND4
Other:
- board text added: "12V+"
- board text added: "12V-"
- board text added: "Bot1"
- board text added: "Bot2"
- board text added: "Bot3"
- board text added: "In"
- board text added: "OUT1"
- board text added: "OUT2"
- board text added: "Out"

Commit message: Digital analizer UPDATE
Parts:
- removed U12: W25Q128JVS, Package_SO:SOIC-8_5.3x5.3mm_P1.27mm
- added C18: 100nF, Capacitor_SMD:C_0603_1608Metric, F.Cu at (103.3, 60.6)
- added C19: 100nF, Capacitor_SMD:C_0603_1608Metric, F.Cu at (99.1, 60.6)
- added C20: 100nF, Capacitor_SMD:C_0603_1608Metric, F.Cu at (93.4, 67.2)
- added C21: 100nF, Capacitor_SMD:C_0603_1608Metric, F.Cu at (94.4, 60.6)
- added C22: 100nF, Capacitor_SMD:C_0603_1608Metric, F.Cu at (92.7, 69.8)
- added J30: Analizador, Connector_PinHeader_2.54mm:PinHeader_2x05_P2.54mm_Vertical, F.Cu at (91.8, 45.2)
- added J31: BOT, Connector_PinHeader_2.54mm:PinHeader_1x04_P2.54mm_Vertical, F.Cu at (135.7, 67.1)
- added J32: UART2_IN, Connector_PinHeader_1.27mm:PinHeader_1x02_P1.27mm_Vertical, F.Cu at (112.4, 73.1)
- added J43: UART_IN, Connector_PinHeader_1.27mm:PinHeader_1x02_P1.27mm_Vertical, F.Cu at (82.2, 76.4)
- added J44: SPI_IN, Connector_PinHeader_1.27mm:PinHeader_1x04_P1.27mm_Vertical, F.Cu at (82.1, 68.5)
- added J45: UART1_IN, Connector_PinHeader_1.27mm:PinHeader_1x02_P1.27mm_Vertical, F.Cu at (112.4, 70.5)
- added J46: RS1_OUT, Connector_PinHeader_1.27mm:PinHeader_1x02_P1.27mm_Vertical, F.Cu at (112.4, 66.6)
- added Q19: BSS138, Package_TO_SOT_SMD:SOT-23, F.Cu at (101.0, 79.0)
- added Q21: BSS138, Package_TO_SOT_SMD:SOT-23, F.Cu at (95.8, 78.8)
- added Q22: BSS138, Package_TO_SOT_SMD:SOT-23, F.Cu at (92.0, 79.0)
- added R83: 5.1k, Resistor_SMD:R_0603_1608Metric, F.Cu at (133.2, 48.2)
- added R84: 5.1k, Resistor_SMD:R_0603_1608Metric, F.Cu at (124.4, 50.3)
- added R85: 1k, Resistor_SMD:R_0603_1608Metric, F.Cu at (100.2, 76.1)
- added R86: 1k, Resistor_SMD:R_0603_1608Metric, F.Cu at (96.6, 76.1)
- added R87: 1k, Resistor_SMD:R_0603_1608Metric, F.Cu at (92.7, 76.1)
- J28: value USB_C_Receptacle_USB2.0_16P -> ANALIZADOR_IN; footprint Connector_USB:USB_C_Receptacle_GCT_USB4105-xx-A_16P_TopMnt_Horizontal -> Connector_PinHeader_1.27mm:PinHeader_1x08_P1.27mm_Vertical
- J29: value Analizador -> SPI
- J36: value SPI -> RS2_OUT; footprint Connector_PinHeader_2.54mm:PinHeader_1x04_P2.54mm_Vertical -> Connector_PinHeader_1.27mm:PinHeader_1x02_P1.27mm_Vertical
- J38: value IN -> POWER
- J41: value SPI -> SPI_OUT
- J42: value UART -> UART_OUT
- SW1: value SW_Push -> BOOT
- SW2: value SW_Push -> RESET
- U4: value RP2040 -> MAX232; footprint Package_DFN_QFN:QFN-56-1EP_7x7mm_P0.4mm_EP3.2x3.2mm -> Package_SO:SOIC-16_4.55x10.3mm_P1.27mm
- moved J29 58.9 mm to (148.9, 67.1)
- moved J36 38.7 mm to (112.4, 78.4), turned to 180 degrees
- moved J28 23.8 mm to (101.5, 57.9)
- moved U4 6.86 mm to (99.1, 67.0)
- moved J40 0.87 mm to (109.0, 61.6)
- moved R77 0.76 mm to (172.6, 43.3)
- moved C16 0.23 mm to (90.3, 64.3)
- moved D14 0.23 mm to (92.4, 63.2)
- moved C15 0.23 mm to (90.2, 61.2)
- moved U22 0.23 mm to (85.0, 63.0)
Connections:
- C16 pad 1: Net-(D14-A) -> /Analizador/Adaptacion/Anal_3.3V
- D14 pad 2: Net-(D14-A) -> /Analizador/Adaptacion/Anal_3.3V
- J29 pad 1: unconnected-(J29-Pin_1-Pad1) -> Net-(J29-Pin_1)
- J29 pad 2: unconnected-(J29-Pin_2-Pad2) -> Net-(J29-Pin_2)
- J29 pad 3: unconnected-(J29-Pin_3-Pad3) -> Net-(J29-Pin_3)
- J29 pad 4: unconnected-(J29-Pin_4-Pad4) -> Net-(J29-Pin_4)
- J29 pad 5: unconnected-(J29-Pin_5-Pad5) -> Net-(J29-Pin_5)
- J29 pad 6: unconnected-(J29-Pin_6-Pad6) -> Net-(J29-Pin_6)
- J29 pad 7: unconnected-(J29-Pin_7-Pad7) -> Net-(J29-Pin_7)
- J29 pad 8: unconnected-(J29-Pin_8-Pad8) -> Net-(J29-Pin_8)
- J36 pad 1: unconnected-(J36-Pin_1-Pad1) -> /Analizador/RS_Rx2
- J36 pad 2: unconnected-(J36-Pin_2-Pad2) -> /Analizador/RS_Tx2
- J39 pad A5: unconnected-(J39-CC1-PadA5) -> Net-(J39-CC1)
- J39 pad B5: unconnected-(J39-CC2-PadB5) -> Net-(J39-CC2)
- J41 pad 1: unconnected-(J41-Pin_1-Pad1) -> /Analizador/Adaptacion/CS_in
- J41 pad 2: unconnected-(J41-Pin_2-Pad2) -> Net-(J41-Pin_2)
- J41 pad 3: unconnected-(J41-Pin_3-Pad3) -> /Analizador/Adaptacion/MISO_in
- J41 pad 4: unconnected-(J41-Pin_4-Pad4) -> Net-(J41-Pin_4)
- J42 pad 1: unconnected-(J42-Pin_1-Pad1) -> Net-(J42-Pin_1)
- J42 pad 2: unconnected-(J42-Pin_2-Pad2) -> /Analizador/Adaptacion/Rx_in
- R16 pad 2: unconnected-(R16-Pad2) -> /Analizador/Adaptacion/Anal_3.3V
- R17 pad 2: unconnected-(R17-Pad2) -> /Analizador/Adaptacion/Anal_3.3V
- R23 pad 2: unconnected-(R23-Pad2) -> /Analizador/Adaptacion/Anal_3.3V
- R24 pad 2: unconnected-(R24-Pad2) -> /Analizador/Adaptacion/Anal_3.3V
- R72 pad 2: unconnected-(R72-Pad2) -> /Analizador/Adaptacion/Anal_3.3V
- R73 pad 2: unconnected-(R73-Pad2) -> /Analizador/Adaptacion/Anal_3.3V
- R74 pad 2: unconnected-(R74-Pad2) -> /Analizador/Adaptacion/Anal_3.3V
- R75 pad 2: unconnected-(R75-Pad2) -> /Analizador/Adaptacion/Anal_3.3V
- U22 pad 2: Net-(D14-A) -> /Analizador/Adaptacion/Anal_3.3V
- U23 pad 10: unconnected-(U23-MISO-Pad10) -> Net-(J29-Pin_1)
- U23 pad 11: unconnected-(U23-GPIO9-Pad11) -> Net-(J29-Pin_4)
- U23 pad 12: unconnected-(U23-GPIO10-Pad12) -> Net-(J29-Pin_3)
- U23 pad 13: unconnected-(U23-MOSI-Pad13) -> Net-(J29-Pin_6)
- U23 pad 14: unconnected-(U23-SCLK-Pad14) -> Net-(J29-Pin_5)
- U23 pad 20: unconnected-(U23-GPIO5-Pad20) -> Net-(J31-Pin_3)
- U23 pad 4: unconnected-(U23-GPIO16-Pad4) -> Net-(J29-Pin_7)
- U23 pad 5: unconnected-(U23-GPIO14-Pad5) -> Net-(J29-Pin_8)
- U23 pad 6: unconnected-(U23-GPIO12-Pad6) -> Net-(J31-Pin_2)
- U23 pad 7: unconnected-(U23-GPIO13-Pad7) -> Net-(J31-Pin_1)
- U23 pad 9: unconnected-(U23-CS0-Pad9) -> Net-(J29-Pin_2)
- U4 pad 1: Net-(U4-IOVDD-Pad1) -> Net-(U4-C1+)
- U4 pad 10: Net-(U4-IOVDD-Pad1) -> /Analizador/UART_Tx2
- U4 pad 11: unconnected-(U4-GPIO8-Pad11) -> /Analizador/UART_Tx1
- U4 pad 12: unconnected-(U4-GPIO9-Pad12) -> /Analizador/UART_Rx1
- U4 pad 13: unconnected-(U4-GPIO10-Pad13) -> /Analizador/RS_Rx1
- U4 pad 14: unconnected-(U4-GPIO11-Pad14) -> /Analizador/RS_TX1
- U4 pad 15: unconnected-(U4-GPIO12-Pad15) -> GND6
- U4 pad 16: unconnected-(U4-GPIO13-Pad16) -> Net-(J40-Pin_2)
- U4 pad 2: unconnected-(U4-GPIO0-Pad2) -> Net-(U4-VS+)
- U4 pad 3: unconnected-(U4-GPIO1-Pad3) -> Net-(U4-C1-)
- U4 pad 4: unconnected-(U4-GPIO2-Pad4) -> Net-(U4-C2+)
- U4 pad 5: unconnected-(U4-GPIO3-Pad5) -> Net-(U4-C2-)
- U4 pad 6: unconnected-(U4-GPIO4-Pad6) -> Net-(U4-VS-)
- U4 pad 7: unconnected-(U4-GPIO5-Pad7) -> /Analizador/RS_Tx2
- U4 pad 8: unconnected-(U4-GPIO6-Pad8) -> /Analizador/RS_Rx2
- U4 pad 9: unconnected-(U4-GPIO7-Pad9) -> /Analizador/UART_Rx2
Routing:
- net GND6: track 0.00 -> 178.3 mm, vias 0 -> 1
- net /Analizador/Adaptacion/Anal_3.3V: track 0.00 -> 73.6 mm, vias 0 -> 2
- net Net-(D13-A): track 37.2 -> 102.9 mm, vias 0 -> 4
- net /Centro_control/TTL-USB/Rx: track 0.00 -> 53.6 mm, vias 0 -> 2
- net Net-(J31-Pin_2): track 0.00 -> 53.1 mm, vias 0 -> 2
- net /Centro_control/TTL-USB/Tx: track 0.00 -> 52.3 mm, vias 0 -> 2
- net Net-(J31-Pin_1): track 0.00 -> 51.7 mm, vias 0 -> 2
- net GND5: track 168.9 -> 208.1 mm
- net Net-(J31-Pin_3): track 0.00 -> 38.4 mm, vias 0 -> 1
- net EN: track 9.30 -> 43.7 mm, vias 0 -> 1
- net Net-(J29-Pin_7): track 0.00 -> 28.0 mm, vias 0 -> 1
- net Net-(J41-Pin_4): track 0.00 -> 25.9 mm
- net /Analizador/Adaptacion/MISO_out: track 0.00 -> 25.4 mm
- net PROG: track 18.2 -> 43.6 mm, vias 0 -> 1
- net Net-(J40-Pin_2): track 0.00 -> 25.2 mm
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- added copper zone on B.Cu, net GND5
- added copper zone on F.Cu, net GND5
- added copper zone on B.Cu, net GND6
- added copper zone on F.Cu, net GND6
Other:
- board text added: "Boton_1"
- board text added: "Boton_2"
- board text added: "Boton_3"
- board text added: "CS0 MISO"
- board text added: "CS2 CS1"
- board text added: "CS4 CS3"
- board text added: "In1"
- board text added: "In2"
- board text added: "In3"
- board text added: "In4"
- board text added: "In5"
- board text added: "In6"
- board text added: "In7"
- board text added: "In8"
- board text added: "Logic analizer and sniffer rp2040 Luis Miguel Carmona Cortés"
- board text added: "MOSI SCLK"
- board text added: "Main control station ESP12F Luis Miguel Carmona Cortés"
- board text added: "Out1"
- board text added: "Out2"
- board text added: "Out3"
- board text added: "Out4"
- board text added: "Out5"
- board text added: "Out6"
- board text added: "Out7"
- board text added: "Out8"
- board text added: "Rx"
- board text added: "Select voltage ch32v006 Luis Miguel Carmona Cortés"
- board text added: "Tx"
