File: Tec/HW_Laboratory/Laboratory/Laboratory.kicad_pcb (KiCad board)
At the start: 2 copper layers, 99.3 x 99.6 mm, 235 parts, among them J1 ENTRADA, J10 SPI, J11 A0, J12 A1, J13 I2C, J14 CON1, J15 I2C, J16 CONTROL, J17 PROG, J18 AUX, J19 BOT, J2 SALIDA, J20 OUT, J21 Pot3, J22 PROG, J23 BOT, J24 I2C, J25 POWER, J26 Pot1, J27 Pot2, J28 ANALIZADOR_IN, J29 SPI, J3 IN, J30 Analizador, J31 BOT, J32 UART2_IN, J33 Pot6, J34 Pot4, J35 Pot5, J36 RS2_OUT, J37 UART, J38 POWER, J39 USB_C_Receptacle_USB2.0_16P, J4 CONTROL, J40 POWER, J41 SPI_OUT, J42 UART_OUT, J43 UART_IN, J44 SPI_IN, J45 UART1_IN, J46 RS1_OUT, J5 OUT, J6 A2, J7 A0, J8 A2, J9 A1, Q1 AO3401A, Q10 BSS138, Q11 BSS138, Q12 BSS138, Q13 BSS138, Q14 BSS138, Q15 BSS138, Q16 BSS138, Q17 BSS138, Q18 BC547, Q19 BSS138, Q2 BC847BS, Q20 BC547, Q21 BSS138, Q22 BSS138, Q3 AO3401A, Q4 BC847BS, Q5 AO3401A, Q6 AO3401A, Q7 BC847BS, Q8 AO3401A, Q9 AO3401A, SW1 BOOT, SW2 RESET, U1 LM2596S-ADJ, U10 LM75B, U11 ch32v006k8u6, U13 LM358, U14 74HC595, U15 CH32V003AxMx, U16 AT24CS32-SSHM, U19 74HC595, U2 MT3608, U20 LM358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

Commit message: Laboratory v2.0:Update the PCB and the Software
Parts:
- removed C17: 100nF, Capacitor_SMD:C_0603_1608Metric
- removed D10, D11, D12, D8, D9: BZX84Cxx, Package_TO_SOT_SMD:SOT-23
- removed J39: USB_C_Receptacle_USB2.0_16P, Connector_USB:USB_C_Receptacle_GCT_USB4105-xx-A_16P_TopMnt_Horizontal
- removed J6, J8: A2, Connector_PinHeader_1.00mm:PinHeader_1x03_P1.00mm_Vertical
- removed Q18, Q20: BC547, Package_TO_SOT_THT:TO-92_Inline
- removed R27, R28, R79, R80: 10k, Resistor_SMD:R_0603_1608Metric
- removed R83, R84: 5.1k, Resistor_SMD:R_0603_1608Metric
- removed U25: CH340C, Package_SO:SOIC-16_3.9x9.9mm_P1.27mm
- added C23: 100nF, Capacitor_SMD:C_0603_1608Metric, F.Cu at (144.6, 113.3)
- added C24: 100nF, Capacitor_SMD:C_0603_1608Metric, F.Cu at (142.0, 117.0)
- added J47: GEN, Connector_PinHeader_2.54mm:PinHeader_1x04_P2.54mm_Vertical, F.Cu at (142.6, 121.6)
- added J48: REGs, Connector_PinHeader_2.54mm:PinHeader_1x03_P2.54mm_Vertical, F.Cu at (121.7, 103.3)
- added J49: Regx, Connector_PinHeader_2.54mm:PinHeader_1x01_P2.54mm_Vertical, F.Cu at (91.7, 88.2)
- added J50: I2C, Connector_PinHeader_2.54mm:PinHeader_1x02_P2.54mm_Vertical, F.Cu at (133.2, 103.4)
- added R81: 100, Resistor_SMD:R_0603_1608Metric, F.Cu at (145.2, 115.7)
- added R82: 10k, Resistor_SMD:R_0603_1608Metric, F.Cu at (149.0, 114.9)
- added R88: 10k, Resistor_SMD:R_0603_1608Metric, F.Cu at (146.2, 118.1)
- added U17: MCP1700x-120xxTT, Package_TO_SOT_SMD:SOT-23, F.Cu at (125.8, 63.5)
- added U18: ch32v006k8u6, Package_DFN_QFN:QFN-32-1EP_4x4mm_P0.4mm_EP2.65x2.65mm, F.Cu at (129.7, 49.4)
- C1: footprint Capacitor_SMD:C_Elec_5x5.4 -> Capacitor_SMD:CP_Elec_6.3x5.4
- C2: footprint Capacitor_SMD:C_Elec_5x5.4 -> Capacitor_SMD:CP_Elec_8x10
- C3, C4: footprint Capacitor_SMD:C_0603_1608Metric -> Capacitor_SMD:C_0805_2012Metric
- D7: value BZX84Cxx -> LED; footprint Package_TO_SOT_SMD:SOT-23 -> LED_SMD:LED_0603_1608Metric
- J11, J12, J7, J9: footprint Connector_PinHeader_1.00mm:PinHeader_1x03_P1.00mm_Vertical -> Connector_PinHeader_1.00mm:PinHeader_1x03_P1.00mm_Vertical_SMD_Pin1Left
- Q6: value AO3401A -> BC847BS; footprint Package_TO_SOT_SMD:SOT-23 -> Package_TO_SOT_SMD:SOT-363_SC-70-6
- Q7: value BC847BS -> 2N7002; footprint Package_TO_SOT_SMD:SOT-363_SC-70-6 -> Package_TO_SOT_SMD:SOT-23
- U24: value AMS1117-3.3 -> LM75B; footprint Package_TO_SOT_SMD:SOT-223-3_TabPin2 -> Package_SO:SOIC-8_3.9x4.9mm_P1.27mm
- U7: value LM75B -> MCP1700x-120xxTT; footprint Package_SO:SOIC-8_3.9x4.9mm_P1.27mm -> Package_TO_SOT_SMD:SOT-23
- moved U24 65.0 mm to (151.2, 118.5), turned to 0 degrees
- moved Q8 46.5 mm to (87.7, 89.5), turned to -90 degrees
- moved J3 44.7 mm to (84.8, 94.0), turned to -90 degrees
- moved Q9 41.8 mm to (87.0, 122.3), turned to -90 degrees
- moved J4 38.2 mm to (82.0, 103.6), turned to 0 degrees
- moved J31 37.9 mm to (164.3, 42.3)
- moved J11 37.1 mm to (101.4, 126.3), turned to 0 degrees
- moved C1 35.2 mm to (93.3, 95.1), turned to -90 degrees
- moved J12 32.6 mm to (101.4, 122.2), turned to 0 degrees
- moved J13 32.5 mm to (82.0, 120.0), turned to 0 degrees
- moved C14 32.1 mm to (161.2, 67.3), turned to -90 degrees
- moved J14 28.7 mm to (82.0, 112.0), turned to 0 degrees
- moved D7 27.5 mm to (146.3, 113.4), turned to -90 degrees
- moved Q7 26.2 mm to (144.4, 132.8), turned to 0 degrees
- moved D3 24.5 mm to (102.6, 136.2), turned to 180 degrees
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Connections:
- net /Centro_control/TTL-USB/Rx renamed Net-(J37-Pin_3)
- net /Centro_control/TTL-USB/Tx renamed Net-(J37-Pin_2)
- C12 pad 1: /Centro_control/TTL-USB/VUSB -> Net-(J38-Pin_1)
- C3 pad 1: /Fuente_alimentacion/Regulador/Vin -> Net-(Q9-D)
- C6 pad 2: /Fuente_alimentacion/Selector/5V_fixed -> +3.3V
- D7 pad 1: Net-(D7-A) -> GND2
- D7 pad 2: unconnected-(D7-NC-Pad2) -> Net-(D7-A)
- J16 pad 7: /Fuente_alimentacion/Selector/Control/BOOST_2 -> /Fuente_alimentacion/Selector/Control/Tx
- J16 pad 8: /Fuente_alimentacion/Selector/Control/BUCK_2 -> /Fuente_alimentacion/Selector/Control/Rx
- J3 pad 1: /Fuente_alimentacion/Regulador/Vin -> /Fuente_alimentacion/Regulador/Ent
- J38 pad 1: /Centro_control/TTL-USB/VUSB -> Net-(J38-Pin_1)
- L2 pad 1: /Fuente_alimentacion/Regulador/Vin -> Net-(Q9-D)
- Q1 pad 1: Net-(D7-A) -> Net-(Q1-G)
- Q1 pad 2: /Fuente_alimentacion/Selector/Mosfets/12V_OUT -> /Fuente_alimentacion/Selector/12V_IN
- Q1 pad 3: /Fuente_alimentacion/Selector/12V_IN -> /Fuente_alimentacion/Selector/Mosfets/12V_OUT
- Q2 pad 6: Net-(D7-A) -> Net-(Q1-G)
- Q3 pad 2: /Fuente_alimentacion/Selector/Mosfets/5V_OUT -> /Fuente_alimentacion/Selector/5V_IN
- Q3 pad 3: /Fuente_alimentacion/Selector/5V_IN -> /Fuente_alimentacion/Selector/Mosfets/5V_OUT
- Q4 pad 2: /Fuente_alimentacion/Selector/Control/3.3V_CTRL -> /Fuente_alimentacion/Selector/Control/REG2_CTRL
- Q4 pad 3: Net-(D10-A) -> Net-(J48-Pin_1)
- Q4 pad 5: /Fuente_alimentacion/Selector/Control/REG1_CTRL -> /Fuente_alimentacion/Selector/Control/REG3_CTRL
- Q4 pad 6: Net-(D9-A) -> Net-(J48-Pin_2)
- Q5 pad 1: Net-(D9-A) -> Net-(Q5-G)
- Q5 pad 2: /Fuente_alimentacion/Selector/Mosfets/3.3V_OUT -> /Fuente_alimentacion/Selector/3.3V_IN
- Q5 pad 3: /Fuente_alimentacion/Selector/3.3V_IN -> /Fuente_alimentacion/Selector/Mosfets/3.3V_OUT
- Q6 pad 1: Net-(D10-A) -> GND2
- Q6 pad 2: /Fuente_alimentacion/Selector/Mosfets/REG1_OUT -> /Fuente_alimentacion/Selector/Control/3.3V_CTRL
- Q6 pad 3: /Fuente_alimentacion/Selector/REG1_IN -> Net-(J48-Pin_3)
- Q7 pad 1: GND2 -> /Fuente_alimentacion/Selector/Control/PWM
- Q7 pad 2: /Fuente_alimentacion/Selector/Control/REG2_CTRL -> GND2
- Q7 pad 3: Net-(D12-A) -> Net-(J47-Pin_4)
- Q8 pad 1: Net-(D11-A) -> Net-(J49-Pin_1)
- Q8 pad 2: /Fuente_alimentacion/Selector/Mosfets/REG2_OUT -> /Fuente_alimentacion/Regulador/Ent
- Q8 pad 3: /Fuente_alimentacion/Selector/REG2_IN -> /Fuente_alimentacion/Regulador/Vin
- Q9 pad 1: Net-(D12-A) -> /Fuente_alimentacion/Regulador/BOOST
- Q9 pad 2: /Fuente_alimentacion/Selector/Mosfets/REG3_OUT -> /Fuente_alimentacion/Regulador/Vin
- Q9 pad 3: /Fuente_alimentacion/Selector/REG3_IN -> Net-(Q9-D)
- R11 pad 1: Net-(D9-A) -> Net-(Q5-G)
- R12 pad 1: Net-(D10-A) -> Net-(J48-Pin_3)
- R12 pad 2: /Fuente_alimentacion/Selector/REG1_IN -> /Fuente_alimentacion/Selector/12V_IN
- R13 pad 1: Net-(D11-A) -> Net-(J48-Pin_2)
- R13 pad 2: /Fuente_alimentacion/Selector/REG2_IN -> /Fuente_alimentacion/Selector/12V_IN
- R14 pad 1: Net-(D12-A) -> Net-(J48-Pin_1)
- R14 pad 2: /Fuente_alimentacion/Selector/REG3_IN -> /Fuente_alimentacion/Selector/12V_IN
- R33 pad 2: /Fuente_alimentacion/Selector/Mosfets/REG1_OUT -> /Fuente_alimentacion/Selector/REG1_IN
- R34 pad 2: /Fuente_alimentacion/Selector/Mosfets/REG2_OUT -> /Fuente_alimentacion/Selector/REG2_IN
- R35 pad 2: /Fuente_alimentacion/Selector/Mosfets/REG3_OUT -> /Fuente_alimentacion/Selector/REG3_IN
- R9 pad 1: Net-(D7-A) -> Net-(Q1-G)
- U10 pad 5: Net-(J8-Pin_2) -> GND1
- U11 pad 17: /Fuente_alimentacion/Selector/5V_fixed -> +3.3V
- U11 pad 2: unconnected-(U11-PA5-Pad2) -> /Fuente_alimentacion/Selector/Control/BUCK_2
- U11 pad 27: /Fuente_alimentacion/Selector/Control/BUCK_2 -> /Fuente_alimentacion/Selector/Control/Rx
- U11 pad 28: /Fuente_alimentacion/Selector/Control/BOOST_2 -> /Fuente_alimentacion/Selector/Control/Tx
- U11 pad 3: unconnected-(U11-PA6-Pad3) -> /Fuente_alimentacion/Selector/Control/BOOST_2
- U11 pad 5: unconnected-(U11-PA0-Pad5) -> Net-(J47-Pin_1)
- U11 pad 6: unconnected-(U11-PA1-Pad6) -> Net-(J47-Pin_2)
- U11 pad 7: unconnected-(U11-PA2-Pad7) -> Net-(J47-Pin_3)
- U11 pad 8: unconnected-(U11-PD0-Pad8) -> /Fuente_alimentacion/Selector/Control/PWM
- U2 pad 5: /Fuente_alimentacion/Regulador/Vin -> Net-(Q9-D)
- U24 pad 1: GND5 -> /Fuente_alimentacion/Selector/SDA
- U24 pad 2: /Centro_control/TTL-USB/VUSB -> /Fuente_alimentacion/Selector/SCL
- U24 pad 3: Net-(D13-A) -> /Fuente_alimentacion/Selector/Control/O.S_3
- U6 pad 12: /Fuente_alimentacion/Selector/Mosfets/REG1_OUT -> /Fuente_alimentacion/Selector/REG1_IN
- U6 pad 15: /Fuente_alimentacion/Selector/Mosfets/REG2_OUT -> /Fuente_alimentacion/Selector/REG2_IN
- U6 pad 2: /Fuente_alimentacion/Selector/Mosfets/REG3_OUT -> /Fuente_alimentacion/Selector/REG3_IN
- U7 pad 1: /Fuente_alimentacion/Selector/SDA -> GND2
- U7 pad 2: /Fuente_alimentacion/Selector/SCL -> +3.3V
- U7 pad 3: /Fuente_alimentacion/Selector/Control/O.S_3 -> /Fuente_alimentacion/Selector/5V_fixed
- U9 pad 5: Net-(J6-Pin_2) -> GND1
Routing:
- net GND5: track 208.1 -> 4.45 mm
- net Net-(D13-A): track 102.9 -> 0.00 mm, vias 4 -> 0
- net /Centro_control/TTL-USB/VUSB: track 56.8 -> 0.00 mm, vias 2 -> 0
- net /Fuente_alimentacion/Selector/Mosfets/REG3_OUT: track 55.2 -> 0.00 mm, vias 2 -> 0
- net Net-(J37-Pin_3): track 53.6 -> 0.00 mm, vias 2 -> 0
- net Net-(J31-Pin_2): track 53.1 -> 0.00 mm, vias 2 -> 0
- net /Fuente_alimentacion/Selector/REG3_IN: track 16.7 -> 69.6 mm, vias 0 -> 2
- net Net-(J37-Pin_2): track 52.3 -> 0.00 mm, vias 2 -> 0
- net /Fuente_alimentacion/Selector/REG2_IN: track 13.2 -> 65.3 mm, vias 0 -> 2
- net Net-(J31-Pin_1): track 51.7 -> 0.00 mm, vias 2 -> 0
- net /Fuente_alimentacion/Selector/Mosfets/REG2_OUT: track 47.6 -> 0.00 mm, vias 4 -> 0
- net EN: track 43.7 -> 0.00 mm, vias 1 -> 0
- net PROG: track 43.6 -> 0.00 mm, vias 1 -> 0
- net /Fuente_alimentacion/Selector/REG1_IN: track 13.8 -> 56.2 mm, vias 0 -> 2
- net GND1: track 155.6 -> 196.3 mm, vias 1 -> 8
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- removed copper zone on F.Cu, net /Fuente_alimentacion/Regulador/OUT_BUCK
- removed copper zone on F.Cu, net /Fuente_alimentacion/Regulador/SW_BOOST
- removed copper zone on F.Cu, net /Fuente_alimentacion/Regulador/Vin
- removed copper zone on F.Cu, net /Fuente_alimentacion/Regulador/Vout_buck
- removed copper zone on B.Cu, net GND1
- removed copper zone on F.Cu, net GND1
- removed copper zone on B.Cu, net GND5
- removed copper zone on F.Cu, net GND5
Other:
- board text added: "5V_f"
- board text added: "A0"
- board text added: "A1"
- board text added: "A2"
- board text added: "BT1"
- board text added: "BT2"
- board text added: "BT3"
- board text added: "PWM"
- board text added: "RX"
- board text added: "Reg1"
- board text added: "Reg2"
- board text added: "Reg3"
- board text added: "Vin"
- board text added: "Voltage Selector ch32v006 Luis Miguel Carmona Cortés"
- board text removed: "BOOST"
- board text removed: "BOTON_1"
- board text removed: "BOTON_2"
- board text removed: "BOTON_3"
- board text removed: "BUCK"
- board text removed: "Boton_1"
- board text removed: "Boton_2"
- board text removed: "Boton_3"
- board text removed: "CS0 MISO"
- board text removed: "CS2 CS1"
- board text removed: "CS4 CS3"
- board text removed: "MOSI SCLK"
- board text removed: "Main control station ESP12F Luis Miguel Carmona Cortés"
- board text removed: "O.S"
- board text removed: "OPC"
- board text removed: "Select voltage ch32v006 Luis Miguel Carmona Cortés"
- board text removed: "VCC"
